File: projects/ADR3350/Ref/DuetReference.sch (EAGLE design)
At the start: 165 parts, among them IC1 74LS74D, J1 EXPANSION, J10 E0 MOT, J11 E0 HEAT, J12 E0 TEMP, J13 2-PIN-350, J14 E1 TEMP, J15 uSDHC, J16 CONN_ALT_HEADER, J19 Z_STOP, J2 FAN2, J20 5V_PS, J23 VIN, J24 GND V_IN, J25 FAN0, J28 Probe, J29 FAN1, J30 PanelDUE, J31 GND V_IN, J32 Y_STOP, J33 X_STOP, J34 E0_STOP, J35 E1_STOP, J36 Z A, J37 SPI0, J39 ESP_COMMS, J5 BED TEMP, J6 E1 MOT, J7 Z B, J8 Y MOT, J9 X MOT, P1 CONN_SD, P2 CONN_LCD, U10 74HC125, U13 74HC32, U2 AP7361C-33E-13, U3 A4403, U5 TMC2660

Commit message: AZR
Parts:
- added C10, C47, C8: 10u, resistor:C-EUC0805
- added C100, C21, C30, C31: 0u47, resistor:C-EUC0805
- added C101, C76, C77, C78: 1u 50V, resistor:C-EUC0805
- added C102, C23, C32, C33: 100u 35V, resistor:CPOL-USD
- added C103, C25, C34, C35: 0u1 50V, resistor:C-EUC0805
- added C104, C11, C16, C27, C36, C37, C46, C48, C49, C50, C51, C52, C54, C61, C62, C64, C67, C69, C70, C71, C72, C9: 0u1, resistor:C-EUC0805
- added C105, C110, C15, C29, C38, C39, C56, C57: 0u01 X7R 10% 50V, resistor:C-EUC0805
- added C106, C108, C109, C114, C115, C116, C117, C118, C119, C120, C121, C122, C123, C86, C87, C89: 1n >50V, resistor:C-EUC0805
- added C111, C40, C42, C43: 2n2, resistor:C-EUC0805
- added C18, C19, C53, C59, C60, C63, C65, C68, C84: 2u2, resistor:C-EUC0805
- added C2: 0u01, resistor:C-EUC0805
- added C44, C45: 10p, resistor:C-EUC0805
- added C66: 4u7, resistor:C-EUC0805
- added C91, C94: 10u 35V, resistor:C-EUC0805
- added D10, D11, D12, D19, D4: (no value), led:LEDCHIPLED_0805
- added D18, D21, D8: DO-219AB, diode:DIODE-SOD123
- added D20, D7: E0 Heat, led:LEDCHIPLED_0805
- added D25, D5: SOD-523F, diode:DIODE-SOD523
- added D6: Bed Heat, led:LEDCHIPLED_0805
- added F1: PPTC Resettable Fuse, SparkFun-Fuses:PPTC_HALF-AMP
- added F2: FAN FUSE, fuse:FUSELITTLEFUSE
- added F3: EXT/STEP FUSE, fuse:FUSELITTLEFUSE
- added F4: BED FUSE, fuse:FUSELITTLEFUSE
- added J21: JTAG, SparkFun-Connectors:CORTEX_DEBUG_PTH
- added J3: 5V V_FAN VIN, SparkFun-Connectors:CONN_03
- added JP1: ERASE, jumper:JP1Q
- added L5, L6: 10uH 100MHz, resistor:L-USL1812
- added L7: 4n7h, resistor:L-USL1812
- added R10, R106, R11, R12, R24, R50, R51, R56, R58, R59, R6, R7, R8, R83, R9, R91, R95: 10K, resistor:R-US_R0805
- added R104: 2K2, resistor:R-US_R0805
- added R107: 100R, resistor:R-US_R0805
- added R13: 1R, resistor:R-US_R0805
- added R19, R21, R53: 4K7 0.1%, resistor:R-US_R0805
- added R20, R23, R97: 180R, resistor:R-US_R0805
- added R28, R29, R38, R39, R40, R41, R89, R90: 22R, resistor:R-US_R0805
- added R33, R35, R44, R45, R46, R47, R93, R94: 0R0501, resistor:R-US_R0805
- added R36, R49, R52: DNP 100K, resistor:R-US_R0805
- added R42, R43, R66, R70, R71, R72, R96: 1K, resistor:R-US_R0805
- added R65, R67, R98: 4K7, resistor:R-US_R0805
- added S1: RESET, switch-omron:10-XX
- added TR1, TR5, TR9: PMV40UN2, adafruit:MOSFET-NREFLOW
- added TR2, TR4, TR8: IPD036N04L, transistor-fet:SPD30P06PTO252
- added U1: ATSAM4E8E, Arduino-DUE-V03:ATSAM4E8E
- added U11: 74S02D, 74xx-us:74S02D
- added U6, U7, U8, U9: TMC2660, TMC2660-Eval_v30:TMC2660
- added X2: CRYSTAL_4PIN, Arduino-DUE-V03:CRYSTAL-3.2-2.5
- C81: value (none) -> 0u01
- C83: value (none) -> DNP 47p
Connections:
- net N$42 renamed SPCK_ESP
- removed net N$3: U5.OB2@1
- removed net N$4: U5.OB1@1
- new net E0_STOP_CONN: D11.C, R59.1
- new net E1_STOP_CONN: D19.C, R95.1
- new net ERASE: JP1.2, U1.PB12/ERASE
- new net MISO: R101.1, U1.PA12/PGMD0/MISO
- new net MOSI: R105.1, U1.PA13/PGMD1/MOSI
- new net N$100: C66.1, R13.1
- new net N$101: C67.1, L6.2, R13.2, U1.VDDPLL
- new net N$102: C2.1, D25.C, R107.2, S1.S, S1.S1
- new net N$103: D4.C, R104.2
- new net N$42: R38.1, R46.2, U7.BRA
- new net N$45: C34.2, U7.VHS
- new net N$46: C36.1, U7.5VOUT
- new net N$49: C38.1, R38.2, U7.SRA
- new net N$50: R28.1, R35.2, U6.BRA
- new net N$51: R29.1, R33.2, U6.BRB
- new net N$52: C29.1, R29.2, U6.SRB
- new net N$53: C25.2, U6.VHS
- new net N$54: C27.1, U6.5VOUT
- new net N$57: C15.1, R28.2, U6.SRA
- new net N$58: R40.1, R47.2, U8.BRA
- new net N$59: R41.1, R45.2, U8.BRB
- new net N$60: C57.1, R41.2, U8.SRB
- new net N$61: C35.2, U8.VHS
- new net N$62: C37.1, U8.5VOUT
- new net N$65: C39.1, R40.2, U8.SRA
- new net N$66: R89.1, R94.2, U9.BRA
- new net N$67: R90.1, R93.2, U9.BRB
- new net N$68: C110.1, R90.2, U9.SRB
- new net N$69: C103.2, U9.VHS
- new net N$70: C104.1, U9.5VOUT
- new net N$73: C105.1, R89.2, U9.SRA
- new net N$74: D12.A, R72.1
- new net N$75: D10.A, R70.1
- new net N$76: D11.A, R71.1
- new net N$77: D19.A, R96.1
- new net N$78: R42.2, TR5.G
- new net N$79: R43.2, TR9.G
- new net N$80: R66.2, TR1.G
- new net N$81: R20.2, TR2.G
- new net N$82: D5.C, D6.A, R65.1
- new net N$83: R23.2, TR4.G
- new net N$84: D7.A, R67.1
- new net N$85: R97.2, TR8.G
- new net N$86: D20.A, R98.1
- new net N$87: U11A.O, U11B.I1, U11C.I1, U11D.I1
- new net N$88: F2.2, J3.3
- new net N$89: C65.1, R6.2, U1.PC27/AFE0_AD13
- new net N$90: C10.1, C52.1, C61.1, C62.1, C68.1, C69.1, C70.1, C71.1, C72.1, L6.1, U1.VDDCORE1, U1.VDDCORE2, U1.VDDCORE3, U1.VDDCORE4, U1.VDDCORE5, U1.VDDCORE6, U1.VDDOUT
- new net N$91: C63.1, R7.2, U1.PC31/AFE0_AD11
- new net N$92: C60.1, R8.2, U1.PC30/AFE0_AD10
- new net N$93: C59.1, R9.2, U1.PC29/AFE0_AD9
- new net N$94: C53.1, R10.2, U1.PC12//AFE0_AD8
- new net N$95: C18.1, R11.2, U1.PC15/AFE0_AD7
- new net N$96: C19.1, R12.2, U1.PC13/AFE0_AD6
- new net N$97: C84.1, R50.2, U1.PA18/PGMD6/AFE0_AD1
- new net N$98: C45.1, U1.PB9/XOUT, X2.C1
- new net N$99: C44.1, U1.PB8/XIN, X2.C2
- new net PB4/TDI: J21.NC/TDI, R36.1, U1.PB4/TDI
- new net PB7/TCK: J21.SWDCLK/TCK, R49.1, R83.1, U1.PB7/TCK
- new net RESET: D25.A, J21.!RESET, R106.1, U1.NRST
- new net SG_TST: J21.SWO/TDO, U1.PB5/TDO
- new net SPCK: R100.1, U1.PA14/PGMD2/SPCK
- new net X_STOP_CONN: D12.C, R56.1
- new net Z_STOP_CONN: D10.C, R58.1
- net +3V3: now also C100.1, C11.1, C16.1, C21.1, C30.1, C31.1, C46.1, C47.1, C48.1, C49.1, C50.1, C51.1, C73.1, C74.1, C8.1, C9.1, J21.VCC, JP1.1, L5.1, L7.1, R106.2, R36.2, R49.2, R51.2, R52.2, R70.2, R71.2, R72.2, R96.2, U1.VDDIN, U1.VDDIO1, U1.VDDIO2, U1.VDDIO3, U1.VDDIO4, U1.VDDIO5, U1.VDDIO6, U1.VDDIO7, U11A.I0, U11A.I1, U6.VCC_IO, U7.VCC_IO, U8.VCC_IO, U9.VCC_IO
- net +5V: now also C54.1, J3.1, U11P.VCC
- net ADC: now also U4.ADC
- net ADVREF: now also C64.1, L5.2, R19.2, R21.2, R53.2, U1.ADVREFP
- net BED-: now also D5.A, D6.C, TR2.S
- net BED_PWM: now also R20.1, U11B.O
- net CS3: now also U1.PC19
- net CS4: now also U1.PC20
- net CS5: now also U1.PA24/PGMD12/RTS1
- net DDM: now also U1.PB10/DDM
- net DDP: now also U1.PB11/DDP
- net E0-: now also D7.C, TR4.S
- net E0_DIR: now also U1.PA1/PGMEN1, U8.DIR
- net E0_EN: now also U1.PC17, U8.!CS
- net E0_MOT_1A: now also C118.1, U8.OA2@1, U8.OA2@3
- net E0_MOT_1B: now also C116.1, U8.OA1@1, U8.OA1@3
- net E0_MOT_2A: now also C120.1, U8.OB1@1, U8.OB1@3
- net E0_MOT_2B: now also C122.1, U8.OB2@1, U8.OB2@3
- net E0_PWM: now also R23.1, U11C.O
- net E0_STEP: now also U1.PD5, U8.STEP
- net E0_STOP: now also C43.1, R59.2, U1.PD10
- net E1-: now also D20.C, TR8.S
- net E1_DIR: now also U1.PD9, U9.DIR
- net E1_EN: now also U1.PC25, U9.!CS
- net E1_MOT_1A: now also C119.1, U9.OA2@1, U9.OA2@3
- net E1_MOT_1B: now also C117.1, U9.OA1@1, U9.OA1@3
- net E1_MOT_2A: now also C121.1, U9.OB1@1, U9.OB1@3
- net E1_MOT_2B: now also C123.1, U9.OB2@1, U9.OB2@3
- net E1_PWM: now also R97.1, U11D.O
- net E1_STEP: now also U1.PD4, U9.STEP
- net E1_STOP: now also C111.1, R95.2, U1.PC16
- net E2_DIR: now also U1.PD28
- net E2_EN: now also U1.PD23
- net E2_STEP: now also U1.PD2
- net E2_STOP: now also U1.PE0
- net E3_DIR: now also U1.PD22
- net E3_EN: now also U1.PD24
- net E3_STEP: now also U1.PD1
- net E3_STOP: now also U1.PE1
- net E4_DIR: now also U1.PD16
- net E4_EN: now also U1.PD25
- net E4_STEP: now also U1.PD0
- net E4_STOP: now also U1.PE2
- net E5_DIR: now also U1.PD17
- net E5_EN: now also U1.PD26
- net E5_STEP: now also U1.PD3
- net E5_STOP: now also U1.PE3
- net E6_DIR: now also U1.PC0/AFE0_AD14
- net E6_EN: now also U1.PB14/DAC1
- net E6_STEP: now also U1.PD27
- net E6_STOP: now also U1.PA17/PGMD5/AFE0_AD0
- net ENC_A: now also U1.PA8/PGMM0/XOUT32
- net ENC_B: now also U1.PC7
- net ENC_SW: now also U1.PA7/PGMNVALID/XIN32
- net ENN: now also R51.1, U1.PC6, U6.!EN, U7.!EN, U8.!EN, U9.!EN
- net ESP_3.3VIN: now also L7.2, U4.VCC
- net ESP_DATA_RDY: now also U1.PD31
- net ESP_EN: now also R18.2, U1.PE5, U4.CH_PD
- net ESP_RST: now also R5.2, U1.PE4
- net FAN0: now also R24.2, R42.1, U1.PC23/TIOA4
- net FAN0-: now also D18.A, TR5.D
- net FAN1: now also R43.1, U1.PC26/TIOA4
- net FAN1-: now also D8.A, TR9.D
- net FAN2: now also R66.1, R91.2, U1.PA0/PGMEN0/TIOA0
- net FAN2-: now also D21.A, TR1.D
- net GND: now also C10.2, C100.2, C101.2, C102.-, C104.2, C105.2, C106.2, C108.2, C109.2, C11.2, C110.2, C111.2, C114.2, C115.2, C116.2, C117.2, C118.2, C119.2, C120.2, C121.2, C122.2, C123.2, C15.2, C16.2, C18.2, C19.2, C2.2, C21.2, C23.-, C27.2, C29.2, C30.2, C31.2, C32.-, C33.-, C36.2, C37.2, C38.2, C39.2, C40.2, C42.2, C43.2, C44.2, C45.2, C46.2, C47.2, C48.2, C49.2, C50.2, C51.2, C52.2, C53.2, C54.2, C56.2, C57.2, C59.2, C60.2, C61.2, C62.2, C63.2, C64.2, C65.2, C66.2, C67.2, C68.2, C69.2, C70.2, C71.2, C72.2, C73.2, C74.2, C76.2, C77.2, C78.2, C8.2, C84.2, C86.2, C87.2, C89.2, C9.2, C91.2, C94.2, F1.1, J21.GND@3, J21.GND@5, J21.GNDDTCT, R104.1, R18.1, R24.1, R33.1, R35.1, R44.1, R45.1, R46.1, R47.1, R91.1, R93.1, R94.1, S1.P, S1.P1, TR1.S, TR2.D, TR4.D, TR5.S, TR8.D, TR9.S, U1.GND1, U1.GND2, U1.GND3, U1.GND4, U1.GND5, U1.GND6, U1.GND7, U1.JTAGSEL, U1.TEST, U11P.GND, U6.CLK, U6.GND@1, U6.GND@2, U6.GND@3, U6.TST_MODE, U7.CLK, U7.GND@1, U7.GND@2, U7.GND@3, U7.TST_MODE, U8.CLK, U8.GND@1, U8.GND@2, U8.GND@3, U8.TST_MODE, U9.CLK, U9.GND@1, U9.GND@2, U9.GND@3, U9.TST_MODE, X2.GND@1, X2.GND@2
- net GPIO16: now also U4.GPIO16
- net HEATER0: now also U1.PA19/PGMD7/PWML0, U11B.I0
- net HEATER1: now also U1.PA20/PMGD8/PWML1, U11C.I0
- net HEATER2: now also U1.PA16/PGMD4/PWML2, U11D.I0
- net HEATER3: now also U1.PC3/PWML3
- net HEATER4: now also U1.PC5/TIOA6
- net HEATER5: now also U1.PC8/TIOA7
- net HEATER6: now also U1.PC11/TIOA8
- net HEATER7: now also U1.PA15/PGMD3/TIOA1
- net LCD_DB4: now also U1.PD21
- net LCD_DB5: now also U1.PD20
- net LCD_DB6: now also U1.PD19
- net LCD_DB7: now also U1.PD18
- net LCD_E: now also U1.PA25/PGMD13
- net LCD_RS: now also U1.PC28
- net MCCDA: now also U1.PA28/MCCDA
- net MCCK: now also U1.PA29/MCCK
- net MCDA0: now also U1.PA30/MCDA0
- net MCDA1: now also U1.PA31/MCDA0
- net MCDA2: now also U1.PA26/PGMD14/MCDA2
- net MCDA3: now also U1.PA27/PGMD15/MCDA3
- net MISO_ESP: now also R101.2, U4.GPIO12
- net MOSI_ESP: now also R105.2, U4.GPIO13
- net N$18: now also L1.1
- net N$43: now also R39.1, R44.2, U7.BRB; no longer R101.2, U4.GPIO12
- net N$44: now also C56.1, R39.2, U7.SRB; no longer R105.2, U4.GPIO13
- net NPCS0: now also U1.PA11/PGMM3/NPCS0
- net PB6/TMS: now also J21.SWDIO/TMS, R52.1, U1.PB6/TMS
- net PS_ON: now also U1.PD15
- net PWR_FAIL_DET1: now also U1.PB3/AFE1_AD1
- net PWR_FAIL_DET2: now also U1.PC4/AFE1_AD7
- net RESET_EXT: now also R107.1
- net SAM_TFR_RDY: now also U1.PD30
- net SD_CD: now also U1.PC21
- net SG_TST_E0: now also U8.SG_TST
- net SG_TST_E1: now also U9.SG_TST
- net SG_TST_Y: now also U7.SG_TST
- net SG_TST_Z: now also U6.SG_TST
- net SPI0_CS0: now also U1.PC24/TIOB3
- net SPI0_CS1: now also U1.PB2/CTS0
- net SPI0_CS2: now also U1.PC18
- net SPI0_MISO: now also U1.PB0/RXD0
- net SPI0_MOSI: now also U1.PB1/TXD0
- net SPI0_SCK: now also U1.PB13/SCK0/DAC0
- net SPI1_MISO: now also U1.PA21/PGMD9/RXD1, U6.SDO, U7.SDO, U8.SDO, U9.SDO
- net SPI1_MOSI: now also U1.PA22/PGMD10/TXD1
- net SPI1_MOSI_BUF: now also U6.SDI, U7.SDI, U8.SDI, U9.SDI
- net SPI1_SCK: now also U1.PA23/PGMD11/SCK1
- net SPI1_SCK_BUF: now also U6.SCK, U7.SCK, U8.SCK, U9.SCK
- net THERMISTOR0: now also R12.1, R21.1
- net THERMISTOR1: now also R11.1, R19.1
- net THERMISTOR2: now also R10.1, R53.1
- net THERMISTOR3: now also R9.1
- net THERMISTOR4: now also R8.1
- net THERMISTOR5: now also R7.1
- net THERMISTOR6: now also R6.1
- net THERMISTOR7: now also R50.1
- net TWCK0: now also U1.PA4/PGMNCMD/TWCK0
- net TWD0: now also U1.PA3/TWD0
- net URXD0: now also U1.PA9/PGMM1
- net URXD1: now also U1.PA5/PGMRDY/URXD1
- net USB_PWR_MON: now also U1.PC22
- net UTXD0: now also U1.PA10/PGMM2/UTXD0
- net UTXD1: now also U1.PA6/PGMNOE/UTXD1
- net VSSA: now also F1.2, R83.2
- net V_BED: now also C91.1, F4.2, R65.2
- net V_FAN: now also D18.C, D21.C, D8.C, J3.2
- net V_FUSED: now also C101.1, C102.+, C103.1, C23.+, C25.1, C32.+, C33.+, C34.1, C35.1, C76.1, C77.1, C78.1, C94.1, F3.2, R67.2, R98.2, U6.NC1, U6.NC33, U6.VS, U6.VSA, U6.VSB, U7.NC1, U7.NC33, U7.VS, U7.VSA, U7.VSB, U8.NC1, U8.NC33, U8.VS, U8.VSA, U8.VSB, U9.NC1, U9.NC33, U9.VS, U9.VSA, U9.VSB
- net V_IN: now also F2.1, F3.1, F4.1
- net X_DIR: now also U1.PD11
- net X_EN: now also U1.PD14
- net X_MOT_2A: now also U5.OB1@1
- net X_MOT_2B: now also U5.OB2@1
- net X_STEP: now also U1.PD6
- net X_STOP: now also C40.1, R56.2, U1.PC14
- net Y_DIR: now also U1.PD12, U7.DIR
- net Y_EN: now also U1.PC9, U7.!CS
- net Y_MOT_1A: now also C89.1, U7.OA2@1, U7.OA2@3
- net Y_MOT_1B: now also C86.1, U7.OA1@1, U7.OA1@3
- net Y_MOT_2A: now also C108.1, U7.OB1@1, U7.OB1@3
- net Y_MOT_2B: now also C114.1, U7.OB2@1, U7.OB2@3
- net Y_STEP: now also U1.PD7, U7.STEP
- net Y_STOP: now also U1.PA2
- net Z_DIR: now also U1.PD13, U6.DIR
- net Z_EN: now also U1.PC10, U6.!CS
- net Z_MOT_1A: now also C106.1, U6.OA2@1, U6.OA2@3
- net Z_MOT_1B: now also C87.1, U6.OA1@1, U6.OA1@3
- net Z_MOT_2A: now also C109.1, U6.OB1@1, U6.OB1@3
- net Z_MOT_2B: now also C115.1, U6.OB2@1, U6.OB2@3
- net Z_PROBE_MCU: now also U1.PC1/AFE1_AD4
- net Z_PROBE_MOD: now also U1.PC2
- net Z_PROBE_MOD_BUF: now also D4.A
- net Z_STEP: now also U1.PD8, U6.STEP
- net Z_STOP: now also C42.1, R58.2, U1.PD29
Other:
- note added: "F2 = 1A (optionally 2A)"
- note added: "F3 = 7.5A (optionally 10A)"
- note added: "F4 = 15A"
- moved on the sheet: C107, C113, C14, C20, C22, C24, C26, C28, C41, C73, C74, C75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
