File: projects/AZR3350/V1/AZR3350.sch (EAGLE design)
At the start: 130 parts, among them IC1 LM2734Y, IC2 LDO-TS1117CW-3V3, IC3 SAMD21G18A-AUT, IC4 MCP23008, IC5 A4988, IC6 A4988, IC7 A4988, IC8 A4988, IC9 SI87XXIS, J107 ZX62-AB-5PA, J2 455-1750-1-ND, J3 455-1750-1-ND, J4 455-1750-1-ND, Q1 FDS6890A, Q2 IRF520, Q3 IRF520, X1 MSTBA4, X3 MSTBV4

Commit message: AZR-V1
Parts:
- removed IC4: MCP23008, misc:MCP23008
- removed J1: (no value), SparkFun-Connectors:CONN_04SMALL
- removed J10, J7, J8, J9: (no value), SparkFun-Connectors:CONN_04
- removed J11: (no value), SparkFun-Connectors:CONN_05X2PTH
- removed J2, J3, J4: 455-1750-1-ND, SparkFun-Connectors:CONN_03SMALL
- removed J5, J6: (no value), SparkFun-Connectors:CONN_02
- removed R10, R9: 10K, resistor:R-US_R0402
- removed R40: 220R, resistor:R-US_R0402
- removed R41: 10K, resistor:R-TRIMM3103
- removed R7, R8: 4.7K, resistor:R-US_R0402
- added 180R, 4K7: (no value), resistor:R-US_R0402
- added LED3, LED4: (no value), led:LEDCHIPLED_0805
- added X10, X11, X12, X13: KK-254-4, con-other:KK-254-4
- added X14, X15: 057-010-1, con-panduit:057-010-1
- added X2: MSTBA2, con-phoenix-508:MSTBA2
- added X4, X5: KK-254-3, con-other:KK-254-3
- added X6, X7, X8, X9: KK-254-2, con-other:KK-254-2
- X1: value MSTBA4 -> KK-254-3; device con-phoenix-508:MSTBA4 -> con-other:KK-254-3
Connections:
- net N$31 renamed RSTX
- net N$38 renamed REFX-IN
- net N$4 renamed RSTY
- net N$41 renamed RSTZ
- net N$55 renamed RSTE
- net N$65 renamed REFE-IN
- removed net +12V: C1.+, C10.1, C12.1, C13.+, C15.2, C17.1, C19.1, C20.+, C22.2, C24.1, C26.1, C27.+, C29.2, C31.1, C33.1, C34.+, C8.2, IC1.VIN, IC5.VBB1, IC5.VBB2, IC6.VBB1, IC6.VBB2, IC7.VBB1, IC7.VBB2, IC8.VBB1, IC8.VBB2, J5.1, J6.1, L1.2, R1.1, R46.2, SJ2.1, X3-2.1
- removed net N$10: J11.4, R41.S
- removed net N$14: IC6.OUT2B, J8.1
- removed net N$15: IC6.OUT2A, J8.2
- removed net N$16: IC6.OUT1A, J8.3
- removed net N$17: IC6.OUT1B, J8.4
- removed net N$28: IC4./RST, R9.2
- removed net N$29: IC4.A0, IC4.A1, IC4.A2, R10.2
- removed net N$46: IC7.OUT2B, J9.1
- removed net N$47: IC7.OUT2A, J9.2
- removed net N$48: IC7.OUT1A, J9.3
- removed net N$49: IC7.OUT1B, J9.4
- removed net N$5: J11.3, R40.2
- removed net N$6: IC5.OUT2B, J7.1
- removed net N$60: IC8.OUT2B, J10.1
- removed net N$61: IC8.OUT2A, J10.2
- removed net N$62: IC8.OUT1A, J10.3
- removed net N$63: IC8.OUT1B, J10.4
- removed net N$7: IC5.OUT2A, J7.2
- removed net N$8: IC5.OUT1A, J7.3
- removed net N$9: IC5.OUT1B, J7.4
- removed net V_BED: R47.2, X1-1.1, X3-4.1
- new net +24V: C1.+, C10.1, C12.1, C13.+, C15.2, C17.1, C19.1, C20.+, C22.2, C24.1, C26.1, C27.+, C29.2, C31.1, C33.1, C34.+, C8.2, IC1.VIN, IC5.VBB1, IC5.VBB2, IC6.VBB1, IC6.VBB2, IC7.VBB1, IC7.VBB2, IC8.VBB1, IC8.VBB2, L1.2, LED3.A, R1.1, R46.2, SJ2.1, X3-2.1, X6-1.S, X7-1.S
- new net BEEPER: X14-1.S
- new net BTN_EN1: X15-5.S
- new net BTN_EN2: X15-3.S
- new net BTN_ENC: X14-2.S
- new net CARDDETECT: X15-7.S
- new net EMOT1A: IC8.OUT1A, X13-3.S
- new net EMOT1B: IC8.OUT1B, X13-4.S
- new net EMOT2A: IC8.OUT2A, X13-2.S
- new net EMOT2B: IC8.OUT2B, X13-1.S
- new net KILL: X15-10.S
- new net N$33: 4K7.1, LED3.C
- new net N$34: 180R.1, LED4.C
- new net SS: X15-4.S
- new net XMOT1A: IC5.OUT1A, X10-3.S
- new net XMOT1B: IC5.OUT1B, X10-4.S
- new net XMOT2A: IC5.OUT2A, X10-2.S
- new net XMOT2B: IC5.OUT2B, X10-1.S
- new net YMOT1A: IC6.OUT1A, X11-3.S
- new net YMOT1B: IC6.OUT1B, X11-4.S
- new net YMOT2A: IC6.OUT2A, X11-2.S
- new net YMOT2B: IC6.OUT2B, X11-1.S
- new net ZMOT1A: IC7.OUT1A, X12-3.S
- new net ZMOT1B: IC7.OUT1B, X12-4.S
- new net ZMOT2A: IC7.OUT2A, X12-2.S
- new net ZMOT2B: IC7.OUT2B, X12-1.S
- net +3V3: now also LED4.A, X1-2.S, X14-10.S, X4-2.S; no longer IC4.VCC, J11.1, J3.2, J4.2, R41.A, R7.1, R8.1, R9.1
- net +5V: no longer R40.1
- net GND: now also 180R.2, 4K7.2, X1-3.S, X14-9.S, X15-9.S, X2-2.1, X4-3.S, X5-3.S, X8-2.S, X9-2.S; no longer IC4.GND, J1.2, J1.4, J11.2, J2.3, J3.3, J4.3, R10.1, R41.E, X1-2.1, X1-4.1
- net LCD_D4: now also X14-5.S; no longer IC4.GP3, J11.8
- net LCD_D5: now also X14-6.S; no longer IC4.GP4, J11.7
- net LCD_D6: now also X14-7.S; no longer IC4.GP5, J11.6
- net LCD_D7: now also X14-8.S; no longer IC4.GP6, J11.5
- net LCD_E: now also X14-3.S; no longer IC4.GP2, J11.10
- net LCD_RS: now also X14-4.S; no longer IC4.GP1, J11.9
- net MISO: now also X15-1.S
- net MOSI: now also X15-6.S
- net N$12: now also X5-2.S; no longer J2.2
- net N$2: now also X8-1.S; no longer J1.1
- net N$21: now also X7-2.S; no longer J6.2
- net N$22: now also X6-2.S; no longer J5.2
- net N$3: now also X9-1.S; no longer J1.3
- net RESET: now also X15-8.S
- net SCK: now also X15-2.S
- net SCL: no longer IC4.SCL, R7.2
- net SDA: no longer IC4.SDA, R8.2
- net VIN: now also R47.2, X2-1.1, X3-4.1; no longer X1-3.1
- net X_STOP: now also X1-1.S; no longer J4.1
- net Y_STOP: now also X4-1.S; no longer J3.1
- net Z_STOP_IN: now also X5-1.S; no longer J2.1
Other:
- moved on the sheet: LED2, R47
