File: projects/AZR3350/V1/AZR3350.brd (EAGLE design)
At the start: 128 x 80.5 mm, 129 parts, among them IC1 LM2734Y, IC2 LDO-TS1117CW-3V3, IC3 SAMD21G18A-AUT, IC5 A4988, IC6 A4988, IC7 A4988, IC8 A4988, IC9 SI87XXIS, J107 ZX62-AB-5PA, Q1 FDS6890A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

Commit message: 58.4%
Parts:
- removed IC3: SAMD21G18A-AUT, Zero_V1.0:TQFP48
- added U$2: ATSAM4S8C, misc:LQFP100
- added X16: (no value), adafruit:ESP-12
- moved IC9 181.1 mm to (100.3, 67.9)
- moved SJ2 152.7 mm to (84.5, 70.5), turned to 270 degrees
- moved SJ1 150.2 mm to (84.5, 66.7), turned to 90 degrees
- moved Q1 137.6 mm to (50.8, 72.4), turned to 0 degrees
- moved R43 135.6 mm to (52.1, 67.9)
- moved C26 134.2 mm to (63.0, 42.3), turned to 0 degrees
- moved R27 133.9 mm to (60.2, 44.3), turned to 90 degrees
- moved C21 130.6 mm to (58.2, 42.8), turned to 180 degrees
- moved R42 130.5 mm to (48.9, 67.9), turned to 0 degrees
- moved C22 129.3 mm to (58.2, 43.9), turned to 0 degrees
- moved C24 127.1 mm to (63.0, 35.2), turned to 0 degrees
- moved R25 123.1 mm to (53.6, 38.4), turned to 180 degrees
- moved C23 121.2 mm to (50.5, 38.9)
- moved C25 120.4 mm to (57.5, 34.7)
- moved J107 120.0 mm to (17.8, 75.6), turned to 180 degrees
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Connections:
- removed net AREF: IC3.4
- removed net RXD: IC3.38
- removed net RX_LED: IC3.48
- removed net SCL: IC3.32
- removed net SDA: IC3.31
- removed net TXD: IC3.37
- removed net TX_LED: IC3.39
- new net VCC: X16.8
- net +3V3: no longer IC3.17, IC3.36, IC3.44
- net ADVREF: no longer IC3.6
- net BED: no longer IC3.13
- net E_DIR: no longer IC3.28
- net E_EN: no longer IC3.30
- net E_STEP: no longer IC3.29
- net FAN1: no longer IC3.23
- net FAN2: no longer IC3.22
- net GND: now also X16.9; no longer IC3.18, IC3.35, IC3.42, IC3.5
- net HOTEND: no longer IC3.14
- net MISO: no longer IC3.21
- net MOSI: no longer IC3.19
- net RESET: no longer IC3.40
- net SCK: no longer IC3.20
- net T_BED: no longer IC3.47
- net T_EXT: no longer IC3.3
- net USB_N: no longer IC3.33
- net USB_P: no longer IC3.34
- net VDDCORE: no longer IC3.43
- net XIN32: no longer IC3.1
- net XOUT32: no longer IC3.2
- net X_DIR: no longer IC3.7
- net X_EN: no longer IC3.9
- net X_STEP: no longer IC3.8
- net X_STOP: no longer IC3.15
- net Y_DIR: no longer IC3.10
- net Y_EN: no longer IC3.12
- net Y_STEP: no longer IC3.11
- net Y_STOP: no longer IC3.16
- net Z_DIR: no longer IC3.25
- net Z_EN: no longer IC3.27
- net Z_STEP: no longer IC3.26
- net Z_STOP: no longer IC3.24
Routing:
- net GND: track 0.00 -> 179.2 mm, vias 9 -> 62
- net +3V3: track 0.00 -> 179.0 mm, vias 0 -> 15
- net +24V: track 113.9 -> 254.1 mm, vias 4 -> 17
- net Z_STOP_IN: track 0.00 -> 19.6 mm
- net N$22: track 0.00 -> 16.2 mm
- net REFZ: track 0.00 -> 12.5 mm
- net REFX: track 0.00 -> 11.0 mm
- net RSTX: track 0.00 -> 9.54 mm
- net N$12: track 0.00 -> 8.84 mm
- net RSTZ: track 0.00 -> 6.78 mm
- net REFY: track 0.00 -> 6.33 mm
- net RSTY: track 0.00 -> 6.12 mm
- net N$21: track 0.00 -> 5.60 mm
- net VREGZ: track 0.00 -> 5.39 mm
- net +5V: track 16.1 -> 11.5 mm
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- added copper zone on layer 1, net +3V3
- added copper zone on layer 16, net +3V3

Commit message: More AZR development; will be changing board shape slightly
Parts:
- added IC10: ATSAM4S8B, misc:LQFP64
- moved U$1 151.0 mm to (109.9, 76.2), turned to 0 degrees
- moved R46 139.5 mm to (86.0, 5.46), turned to 0 degrees
- moved R45 137.7 mm to (94.2, 4.32), turned to 0 degrees
- moved LED1 135.6 mm to (82.5, 5.46), turned to 90 degrees
- moved R47 134.4 mm to (94.2, 5.46)
- moved LED2 133.7 mm to (90.8, 5.46), turned to 90 degrees
- moved R44 126.0 mm to (74.5, 5.46)
- moved X3 1.90 mm to (88.9, 10.2)
Connections:
- new net BEEP: U$2.30
- new net ENC_B: U$2.40
- new net ENC_SW: U$2.49
- new net HEATER0: U$2.25
- new net HEATER1: U$2.47
- new net LCD_CS: U$2.62
- new net N$5: U$2.27, U$2.50, U$2.69, U$2.91, U$2.98
- new net N$6: U$2.16, U$2.36, U$2.56, U$2.85
- new net NPCS0: U$2.42
- new net NRST: U$2.60
- new net SD_CD: U$2.58
- new net THERMISTOR0: U$2.24
- new net THERMISTOR1: U$2.3
- new net TWCK0: U$2.55
- new net URXD1: U$2.7
- new net UTXD1: U$2.9
- net E_STEP: now also U$2.37
- net GND: now also U$2.2, U$2.26, U$2.45, U$2.61, U$2.70, U$2.95
- net MISO: now also U$2.41
- net MOSI: now also U$2.33
- net SCK: now also U$2.31
- net X_STOP: now also U$2.34
- net Y_DIR: now also U$2.48
- net Y_STEP: now also U$2.43
- net Z_DIR: now also U$2.51
- net Z_STEP: now also U$2.54
- net Z_STOP: now also U$2.65
Routing:
- net GND: track 179.2 -> 207.4 mm, vias 62 -> 82
- net +24V: track 254.1 -> 264.2 mm, vias 17 -> 14
- net N$24: track 0.00 -> 5.40 mm
- net VIN: track 17.3 -> 22.7 mm
- net N$23: track 7.03 -> 11.0 mm
- net N$27: track 0.00 -> 1.73 mm
- net N$26: track 0.00 -> 1.73 mm
- net +3V3: track 179.0 -> 177.4 mm
