File: projects/AZR3350/V4/AZR3350.brd (EAGLE design)
At the start: 80.5 x 141.4 mm, 194 parts, among them IC1 LM2734Y, IC10 A4988, IC2 LDO-TS1117CW-3V3, IC3 ATSAM4S8C, IC4 SI87XXIS, IC5 74HC125, IC6 74S08D, IC7 A4988, IC8 A4988, IC9 A4988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

Commit message: Progress...
Parts:
- moved C9 178.8 mm to (146.3, 78.9)
- moved SJ2 30.3 mm to (160.2, 110.1), turned to 90 degrees
- moved SJ1 27.0 mm to (162.8, 110.1), turned to 90 degrees
- moved X_STOP 16.5 mm to (167.4, 132.2)
- moved Z_STOP 16.5 mm to (167.4, 115.7)
- moved R17 15.3 mm to (121.4, 18.2)
- moved R18 15.3 mm to (121.4, 20.2)
- moved R15 15.2 mm to (121.4, 14.5)
- moved R16 15.2 mm to (121.4, 10.4)
- moved R20 15.2 mm to (121.4, 12.4)
- moved IC4 14.0 mm to (160.0, 116.8)
- moved R19 13.4 mm to (121.4, 22.2), turned to 0 degrees
- moved L5 0.80 mm to (117.5, 27.3), turned to 90 degrees
- moved C22 0.63 mm to (133.6, 61.9)
Routing:
- net +3V3: track 286.1 -> 478.8 mm, vias 18 -> 23
- net MCDA1: track 0.00 -> 81.0 mm, vias 0 -> 2
- net URXD1: track 0.00 -> 79.6 mm, vias 0 -> 2
- net MCDA2: track 0.00 -> 77.5 mm, vias 0 -> 2
- net ESP_RST: track 0.00 -> 75.3 mm, vias 0 -> 2
- net UTXD1: track 0.00 -> 75.1 mm, vias 0 -> 2
- net SD_CD: track 0.00 -> 72.9 mm, vias 0 -> 2
- net MCDA0: track 0.00 -> 70.5 mm, vias 0 -> 2
- net NPCS0: track 0.00 -> 69.2 mm, vias 0 -> 2
- net LCD_SCK: track 30.8 -> 98.4 mm, vias 2 -> 4
- net ESP_EN: track 0.00 -> 67.5 mm, vias 0 -> 2
- net MCCDA: track 0.00 -> 66.8 mm, vias 0 -> 2
- net MCCK: track 0.00 -> 65.1 mm, vias 0 -> 2
- net X_STOP: track 0.00 -> 64.1 mm
- net MCDA3: track 0.00 -> 63.0 mm, vias 0 -> 2
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
Commit message: More progress...
Parts:
- moved RESET 183.4 mm to (154.9, 89.3), turned to 180 degrees
- moved R14 177.9 mm to (147.3, 86.6)
- moved C28 175.5 mm to (147.3, 88.6), turned to 180 degrees
- moved R12 158.7 mm to (113.9, 69.6)
- moved C15 156.4 mm to (111.4, 70.6), turned to 180 degrees
- moved ERASE 155.7 mm to (138.6, 84.5), turned to 90 degrees
- moved F1 154.5 mm to (111.6, 67.3)
- moved R37 134.8 mm to (120.9, 98.8)
- moved R36 130.7 mm to (118.9, 98.8)
- moved C8 113.6 mm to (111.4, 96.1)
- moved R11 109.1 mm to (109.3, 96.1)
- moved R10 104.6 mm to (107.3, 96.1), turned to 90 degrees
- moved EXT_L 18.3 mm to (118.1, 109.3), turned to 90 degrees
- moved R42 17.0 mm to (119.8, 107.1)
- moved R46 10.0 mm to (150.4, 59.3), turned to 270 degrees
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Routing:
- net PWR_FAIL_DET: track 0.00 -> 80.9 mm, vias 0 -> 2
- net LCD_SD_CS: track 9.73 -> 67.8 mm, vias 0 -> 2
- net USB_PWR_MON: track 0.00 -> 53.3 mm, vias 0 -> 2
- net LCD_CS: track 0.00 -> 52.9 mm, vias 0 -> 2
- net LCD_MOSI: track 44.3 -> 95.4 mm, vias 2 -> 4
- net HOTEND: track 0.00 -> 51.2 mm, vias 0 -> 2
- net +3V3: track 478.8 -> 523.6 mm, vias 23 -> 26
- net BED: track 0.00 -> 42.6 mm, vias 0 -> 2
- net GND: track 292.7 -> 333.6 mm, vias 65 -> 81
- net RESET: track 0.00 -> 31.9 mm, vias 0 -> 2
- net VSSA: track 0.00 -> 30.4 mm
- net +5V: track 83.1 -> 112.9 mm, vias 2 -> 3
- net BED_G: track 0.00 -> 24.8 mm
- net EXT_D: track 0.00 -> 22.8 mm, vias 0 -> 20
- net BED_D: track 0.00 -> 22.4 mm, vias 0 -> 40
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Other:
- board text added: "Rev. 1.0.4"
- board text removed: "Rev. 1.0.3"

Commit message: Finished, I think
Parts:
- moved C30 0.13 mm to (135.0, 84.5)
Routing:
- net GND: track 333.6 -> 475.0 mm, vias 81 -> 166
- net BEEPER: track 0.00 -> 22.1 mm, vias 0 -> 2
- net VDDOUT: track 57.0 -> 63.6 mm, vias 3 -> 4
- net BOOST: track 0.00 -> 4.02 mm
- net FB: track 0.00 -> 3.77 mm
- net +3V3: track 523.6 -> 526.0 mm, vias 26 -> 30
- net SHDN: track 0.00 -> 1.89 mm
- net USB_PWR_MON: track 53.3 -> 52.2 mm
- net ADVREF: track 11.8 -> 12.9 mm
- net RESET: track 31.9 -> 30.9 mm
- net LCD_MOSI: track 95.4 -> 96.2 mm
- net MCCDA: track 66.8 -> 66.2 mm
- net LCD_SCK: track 99.2 -> 99.8 mm
