File: projects/AZR3350/V4/AZR3350.sch (EAGLE design)
At the start: 194 parts, among them IC1 LM2734Y, IC10 A4988, IC2 LDO-TS1117CW-3V3, IC3 ATSAM4S8C, IC4 SI87XXIS, IC5 74HC125, IC6 74S08D, IC7 A4988, IC8 A4988, IC9 A4988, J1 ZX62-AB-5PA, J3 MSTBV4, J4 MOLEX-105162-001, Q1 NX138BKS, Q2 BUK9Y53-100B, Q3 BUK9Y53-100B, Q4 BC817-16SMD, X1 12MHz

Commit message: Replacing .35mm vias with .4mm
Parts:
- added JP3: (no value), pinhead:PINHD-1X5
- JP1, JP2: device pinhead:PINHD-1X6 -> pinhead:PINHD-1X6/90
Connections:
- removed net LCD_RST: IC3.PC21
- new net LCD_KILL: IC3.PC21, JP3.4
- net +5V: now also JP1.5, JP2.4; no longer JP1.2, JP2.3
- net BTN_EN1: now also JP3.1
- net BTN_EN2: now also JP3.2
- net BTN_ENC: now also JP3.3
- net GND: now also JP1.6, JP3.5; no longer JP1.1
- net LCD_CS_BUF: now also JP1.3; no longer JP1.4
- net LCD_MOSI_BUF: now also JP1.2; no longer JP1.5
- net LCD_SCK_BUF: now also JP1.1; no longer JP1.6
- net N$2: now also JP2.2; no longer JP2.5
- net RESET: now also RESET.P; no longer RESET.P1
Other:
- moved on the sheet: R73

Commit message: New 32-bit AMR3350 (probably will be renamed), + other edits
Connections:
- removed net VIN: D1.A, J3-4.1, PWRIN-1.1, R1.2, R43.2
- new net N$3: C2.+, IC1.VIN, L1.2, R3.1
- net +24V: now also D1.A, J3-4.1, PWRIN-1.1, R1.2, R43.2; no longer C2.+, IC1.VIN, L1.2, R3.1

Commit message: Changes from a while back, which I think involved a different component choice?
Parts:
- removed JP2: (no value), pinhead:PINHD-1X6/90
- removed JP3: (no value), pinhead:PINHD-1X5
- added J2: MOLEX-105162-001, misc:MOLEX-105162-001
- added J5: (no value), con-other:PINHD-1X6
- C37: value 100n -> 1u
- C40, C42, C47, C49, C54, C56, C61, C63: value 220n -> 100n
- C41, C43, C48, C50, C55, C57, C62, C64: value 100n -> 220n
- C44, C51, C58, C65: value 100u -> 100n; device resistor:CPOL-USD -> resistor:C-EUC0603
- C45, C52, C59: value 100n -> 100u; device resistor:C-EUC0603 -> resistor:CPOL-USD
- C66: value 1u -> 100u; device resistor:C-EUC0603 -> resistor:CPOL-USD
- D1: device adafruit:DIODE_SOD-123FL -> diode:SCHOTTKY-DIODESMD
- J4: value MOLEX-105162-001 -> (none); device misc:MOLEX-105162-001 -> con-other:PINHD-1X6
- JP1: device pinhead:PINHD-1X6/90 -> pinhead:PINHD-1X5
- PWRIN: value MSTBA2 -> 2-PIN-508; device con-phoenix-508:MSTBA2 -> con-other:2-PIN-508
- Q2, Q3: value BUK9Y53-100B -> AON7524; device misc:BUK9Y53-100B -> misc:AON7524
- R44: value 10K -> 1K
- R45: value 0R2 -> 47R; device resistor:R-US_R0805 -> resistor:R-US_R0603
- R48, R55, R62, R69: value 100K -> 10K
- R49, R56, R63, R70: value 10K -> 0R2; device resistor:R-TRIMM3103 -> resistor:R-US_R0805
- R50, R57, R64, R71: value 20K -> 100K
- R51, R58, R65: device resistor:R-US_R0603 -> resistor:R-TRIMM3103
- R52, R59, R66: value 0R2 -> 20K; device resistor:R-US_R0805 -> resistor:R-US_R0603
- R72: value 1K -> 10K; device resistor:R-US_R0603 -> resistor:R-TRIMM3103
- R73: value 47R -> 20K
- renumbered ESP8266 to ES1
Connections:
- net +24V: now also C40.2, C42.1, C44.1, C45.+, C47.2, C49.1, C51.1, C52.+, C54.2, C56.1, C58.1, C59.+, C61.2, C63.1, C65.1, C66.+; no longer C39.2, C41.1, C43.1, C44.+, C46.2, C48.1, C50.1, C51.+, C53.2, C55.1, C57.1, C58.+, C60.2, C62.1, C64.1, C65.+
- net +3V3: now also C37.1, C43.1, C50.1, C57.1, C64.1, J2.VDD, R52.2, R59.2, R66.2, R73.2; no longer C42.1, C49.1, C56.1, C63.1, C66.1, J4.VDD, R46.2, R53.2, R60.2, R67.2
- net +5V: now also C38.1, J4.5, J5.4, R45.1; no longer C37.1, JP1.5, JP2.4, R73.1
- net BEEPER: now also R44.1; no longer R72.1
- net BTN_EN1: now also JP1.1; no longer JP3.1
- net BTN_EN2: now also JP1.2; no longer JP3.2
- net BTN_ENC: now also JP1.3; no longer JP3.3
- net CLK: now also J2.CLK; no longer J4.CLK
- net CMD: now also J2.CMD; no longer J4.CMD
- net CP1E: now also C60.1; no longer C59.1
- net CP1X: now also C39.1; no longer C38.1
- net CP1Y: now also C46.1; no longer C45.1
- net CP1Z: now also C53.1; no longer C52.1
- net CP2E: now also C60.2; no longer C59.2
- net CP2X: now also C39.2; no longer C38.2
- net CP2Y: now also C46.2; no longer C45.2
- net CP2Z: now also C53.2; no longer C52.2
- net DAT0: now also J2.DAT0; no longer J4.DAT0
- net DAT1: now also J2.DAT1; no longer J4.DAT1
- net DAT2: now also J2.DAT2; no longer J4.DAT2
- net DAT3: now also J2.DAT3; no longer J4.DAT3
- net DET: now also J2.CARD_DETECT; no longer J4.CARD_DETECT
- net E_EN: now also R69.1; no longer R67.1
- net GND: now also C38.2, C44.2, C45.-, C51.2, C52.-, C58.2, C59.-, C65.2, C66.-, J2.GND, J2.VSS, J4.6, J5.1, J5.6, JP1.5, R46.2, R49.1, R51.E, R53.2, R56.1, R58.E, R60.2, R63.1, R65.E, R67.2, R70.1, R72.E; no longer C40.2, C44.-, C47.2, C51.-, C54.2, C58.-, C61.2, C65.-, C66.2, J4.GND, J4.VSS, JP1.6, JP2.1, JP2.6, JP3.5, R44.2, R45.1, R49.E, R51.2, R52.1, R56.E, R58.2, R59.1, R63.E, R65.2, R66.1, R70.E
- net LCD_CS_BUF: now also J4.3; no longer JP1.3
- net LCD_KILL: now also JP1.4; no longer JP3.4
- net LCD_MOSI_BUF: now also J4.2; no longer JP1.2
- net LCD_SCK_BUF: now also J4.1; no longer JP1.1
- net N$2: now also J5.2, R45.2; no longer JP2.2, R73.2
- net N$7: now also R44.2; no longer R72.2
- net REFE: now also R72.S; no longer R70.S
- net REFE-IN: now also R72.A, R73.1; no longer R70.A, R71.1
- net REFX: now also R51.S; no longer R49.S
- net REFX-IN: now also R51.A, R52.1; no longer R49.A, R50.1
- net REFY: now also R58.S; no longer R56.S
- net REFY-IN: now also R58.A, R59.1; no longer R56.A, R57.1
- net REFZ: now also R65.S; no longer R63.S
- net REFZ-IN: now also R65.A, R66.1; no longer R63.A, R64.1
- net ROSCE: now also R67.1; no longer R65.1
- net ROSCX: now also R46.1; no longer R44.1
- net ROSCY: now also R53.1; no longer R51.1
- net ROSCZ: now also R60.1; no longer R58.1
- net RSTE: now also R71.1; no longer R69.1
- net RSTX: now also R50.1; no longer R48.1
- net RSTY: now also R57.1; no longer R55.1
- net RSTZ: now also R64.1; no longer R62.1
- net SNS1E: now also R68.2; no longer R66.2
- net SNS1X: now also R47.2; no longer R45.2
- net SNS1Y: now also R54.2; no longer R52.2
- net SNS1Z: now also R61.2; no longer R59.2
- net SNS2E: now also R70.2; no longer R68.2
- net SNS2X: now also R49.2; no longer R47.2
- net SNS2Y: now also R56.2; no longer R54.2
- net SNS2Z: now also R63.2; no longer R61.2
- net VCPE: now also C61.1; no longer C60.1
- net VCPX: now also C40.1; no longer C39.1
- net VCPY: now also C47.1; no longer C46.1
- net VCPZ: now also C54.1; no longer C53.1
- net VREGE: now also C62.1; no longer C61.1
- net VREGX: now also C41.1; no longer C40.1
- net VREGY: now also C48.1; no longer C47.1
- net VREGZ: now also C55.1; no longer C54.1
- net X_EN: now also R48.1; no longer R46.1
- net Y_EN: now also R55.1; no longer R53.1
- net Z_EN: now also R62.1; no longer R60.1
Other:
- moved on the sheet: C37, C38, C39, C40, C41, C42, C43, C46, C47, C48, C49, C50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
