File: projects/AMR3350/V6-32/AMR3350.brd (EAGLE design)
At the start: 100 x 87 mm, 244 parts, among them IC1 A4403, IC10 TMC21X0-LA, IC11 TMC21X0-LA, IC12 74LS32D, IC2 LDO-TS1117CW-3V3, IC3 ATSAM4S8C, IC4 SI87XXIS, IC5 74HC125, IC6 74S08D, IC7 TMC21X0-LA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

Commit message: A few small changes
Routing:
- net SG_TST_X: track 81.0 -> 82.3 mm
- net SG_TST_Y: track 62.5 -> 63.7 mm
- net ENN: track 214.9 -> 216.2 mm
- net SG_TST_Z: track 53.3 -> 54.0 mm
- net SG_TST_E1: track 42.3 -> 41.7 mm
Other:
- board text added: "EE4SR3350"
- board text added: "Rev. 1.1.0"

Commit message: Changes from a while back, which I think involved a different component choice?
Parts:
- C40: value 2K2 -> 2.2u
- Q3, Q4: value BUK9Y53-100B -> AON7524; device misc:SOT-669 -> misc:3X3DFN-EP
Connections:
- net EXT1_D: now also Q3.5, Q3.6, Q3.7, Q3.8, Q3.E1, Q3.E2, Q3.PAD; no longer Q3.EXP, Q3.MB
- net EXT2_D: now also Q4.5, Q4.6, Q4.7, Q4.8, Q4.E1, Q4.E2, Q4.PAD; no longer Q4.EXP, Q4.MB
Routing:
- net GND: track 1447.8 -> 1457.1 mm
- net EXT1_G: track 1.84 -> 3.55 mm
- net EXT2_G: track 1.77 -> 3.48 mm
- net EXT2_D: track 21.2 -> 21.3 mm, vias 23 -> 20
- net EXT1_D: track 21.2 -> 21.3 mm, vias 23 -> 20
Other:
- board text added: "-"
Changed lines of the file:
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@@
 <text x="43.815" y="52.705" size="3.81" layer="21" font="vector" ratio="10">EE4SR3350</text>
 <text x="43.815" y="50.8" size="1.016" layer="21" font="vector" ratio="12">Rev. 1.1.0</text>
+<text x="12.7" y="3.81" size="1.778" layer="21" font="vector" ratio="12" rot="R90" align="center">-</text>
 </plain>
 <attributes>
@@
 <attribute name="VALUE" x="79.375" y="49.53" size="1.27" layer="27" rot="R180"/>
 </element>
-<element name="C40" library="resistor" library_urn="urn:adsk.eagle:library:348" package="C0603" package3d_urn="urn:adsk.eagle:package:23616/2" value="2K2" x="62.738" y="1.7145" smashed="yes">
+<element name="C40" library="resistor" library_urn="urn:adsk.eagle:library:348" package="C0603" package3d_urn="urn:adsk.eagle:package:23616/2" value="2.2u" x="62.738" y="1.7145" smashed="yes">
 <attribute name="NAME" x="65.024" y="0.6985" size="0.6096" layer="25" font="vector" ratio="12" rot="R90"/>
 <attribute name="VALUE" x="62.103" y="-0.1905" size="1.27" layer="27"/>
@@
 <attribute name="MF" value="FARNELL" x="-0.635" y="-67.31" size="1.778" layer="27" rot="R270" display="off"/>
 <attribute name="MPN" value="1757242" x="-0.635" y="-67.31" size="1.778" layer="27" rot="R270" display="off"/>
-<attribute name="NAME" x="12.065" y="12.446" size="0.6096" layer="25" font="vector" ratio="12" rot="R270"/>
+<attribute name="NAME" x="0.254" y="12.7" size="0.6096" layer="25" font="vector" ratio="12"/>
 <attribute name="OC_FARNELL" value="3705171" x="-0.635" y="-67.31" size="1.778" layer="27" rot="R270" display="off"/>
 <attribute name="OC_NEWARK" value="71C4161" x="-0.635" y="-67.31" size="1.778" layer="27" rot="R270" display="off"/>
@@
 <attribute name="VALUE" x="11.905" y="48.09" size="1.27" layer="27" rot="R270"/>
 </element>
-<element name="Q3" library="misc" package="SOT-669" value="BUK9Y53-100B" x="26.035" y="26.67" smashed="yes" rot="R90">
-<attribute name="NAME" x="27.432" y="23.876" size="0.6096" layer="25" font="vector" ratio="12" rot="R180"/>
+<element name="Q3" library="misc" package="3X3DFN-EP" value="AON7524" x="26.035" y="26.67" smashed="yes" rot="R90">
+<attribute name="NAME" x="27.432" y="24.511" size="0.6096" layer="25" font="vector" ratio="12" rot="R180"/>
 <attribute name="VALUE" x="31.115" y="24.13" size="1.27" layer="27" rot="R90"/>
 </element>
-<element name="Q4" library="misc" package="SOT-669" value="BUK9Y53-100B" x="26.035" y="36.83" smashed="yes" rot="R90">
-<attribute name="NAME" x="27.559" y="40.132" size="0.6096" layer="25" font="vector" ratio="12" rot="R180"/>
+<element name="Q4" library="misc" package="3X3DFN-EP" value="AON7524" x="26.035" y="36.83" smashed="yes" rot="R90">
+<attribute name="NAME" x="27.559" y="39.497" size="0.6096" layer="25" font="vector" ratio="12" rot="R180"/>
 <attribute name="VALUE" x="31.115" y="34.29" size="1.27" layer="27" rot="R90"/>
 </element>
@@
 <wire x1="57.02845" y1="47.2079875" x2="56.02718125" y2="47.2079875" width="0.3048" layer="1"/>
 <wire x1="57.485" y1="44.705" x2="57.485" y2="46.7514375" width="0.3048" layer="1"/>
-<wire x1="28.76" y1="37.465" x2="30.48" y2="37.465" width="0.6096" layer="1"/>
 <via x="30.48" y="37.465" extent="1-16" drill="0.4"/>
 <via x="30.48" y="36.195" extent="1-16" drill="0.4"/>
 <wire x1="30.48" y1="36.195" x2="30.48" y2="34.925" width="0.6096" layer="1"/>
 <via x="30.48" y="34.925" extent="1-16" drill="0.4"/>
-<wire x1="30.48" y1="34.925" x2="28.76" y2="34.925" width="0.6096" layer="1"/>
-<wire x1="28.76" y1="36.195" x2="30.48" y2="36.195" width="0.6096" layer="1"/>
 <wire x1="30.48" y1="36.195" x2="30.48" y2="37.465" width="0.6096" layer="1"/>
-<wire x1="28.76" y1="27.305" x2="30.48" y2="27.305" width="0.6096" layer="1"/>
 <via x="30.48" y="27.305" extent="1-16" drill="0.4"/>
-<wire x1="28.76" y1="26.035" x2="30.48" y2="26.035" width="0.6096" layer="1"/>
 <via x="30.48" y="26.035" extent="1-16" drill="0.4"/>
-<wire x1="28.76" y1="24.765" x2="30.48" y2="24.765" width="0.6096" layer="1"/>
 <via x="30.48" y="24.765" extent="1-16" drill="0.4"/>
 <wire x1="30.48" y1="24.765" x2="30.48" y2="26.035" width="0.6096" layer="1"/>
@@
 <wire x1="79.9004" y1="25.01073125" x2="79.7782" y2="25.13293125" width="0.254" layer="1"/>
 <wire x1="79.7782" y1="25.13293125" x2="79.7782" y2="25.5522" width="0.254" layer="1"/>
+<wire x1="27.435" y1="37.155" x2="30.17" y2="37.155" width="0.4064" layer="1"/>
+<wire x1="30.17" y1="37.155" x2="30.48" y2="37.465" width="0.4064" layer="1"/>
+<wire x1="27.435" y1="36.505" x2="30.17" y2="36.505" width="0.4064" layer="1"/>
+<wire x1="30.17" y1="36.505" x2="30.48" y2="36.195" width="0.4064" layer="1"/>
+<wire x1="27.435" y1="35.855" x2="29.55" y2="35.855" width="0.4064" layer="1"/>
+<wire x1="29.55" y1="35.855" x2="30.48" y2="34.925" width="0.4064" layer="1"/>
+<wire x1="27.435" y1="26.995" x2="30.17" y2="26.995" width="0.4064" layer="1"/>
+<wire x1="30.17" y1="26.995" x2="30.48" y2="27.305" width="0.4064" layer="1"/>
+<wire x1="27.435" y1="26.345" x2="30.17" y2="26.345" width="0.4064" layer="1"/>
+<wire x1="30.17" y1="26.345" x2="30.48" y2="26.035" width="0.4064" layer="1"/>
+<wire x1="27.435" y1="25.695" x2="29.55" y2="25.695" width="0.4064" layer="1"/>
+<wire x1="29.55" y1="25.695" x2="30.48" y2="24.765" width="0.4064" layer="1"/>
 <wire x1="91.8706" y1="62.308" x2="91.8" y2="62.131" width="0" layer="19" extent="1-1"/>
 <wire x1="72.75" y1="62.131" x2="72.8206" y2="62.308" width="0" layer="19" extent="1-1"/>
@@
 <wire x1="65.405" y1="35.56" x2="65.405" y2="41.275" width="1.27" layer="1"/>
 <wire x1="65.151" y1="41.275" x2="66.167" y2="42.291" width="1.27" layer="1"/>
-<via x="66.167" y="42.291" extent="1-16" drill="0.4"/>
+<via x="66.167" y="42.291" extent="1-16" drill="0.5"/>
 <wire x1="63.5" y1="33.655" x2="65.405" y2="35.56" width="1.27" layer="1"/>
 <wire x1="65.405" y1="35.56" x2="65.643" y2="35.322" width="0.6096" layer="1"/>
@@
 <wire x1="65.96" y1="31.195" x2="65.96" y2="30.02658125" width="0.6096" layer="1"/>
 <wire x1="65.96" y1="30.02658125" x2="65.96" y2="28.955" width="0.3048" layer="1"/>
-<via x="55.245" y="33.655" extent="1-16" drill="0.4"/>
+<via x="55.245" y="33.655" extent="1-16" drill="0.5"/>
 <wire x1="55.245" y1="33.655" x2="62.23" y2="33.655" width="1.27" layer="1"/>
 <wire x1="62.23" y1="33.655" x2="63.373" y2="33.655" width="1.27" layer="1"/>
@@
 <contactref element="J2" pad="1"/>
 <contactref element="EXT1_L" pad="C"/>
-<contactref element="Q3" pad="EXP"/>
-<contactref element="Q3" pad="MB"/>
-<wire x1="25.585" y1="26.67" x2="22.41" y2="23.495" width="1.778" layer="1"/>
-<wire x1="22.41" y1="23.495" x2="5.715" y2="23.495" width="1.778" layer="1"/>
+<contactref element="Q3" pad="5"/>
+<contactref element="Q3" pad="6"/>
 <polygon width="0.1524" layer="1" isolate="0.4064" thermals="no">
 <vertex x="3.175" y="22.225"/>
@@
 <vertex x="27.686" y="22.225"/>
 </polygon>
-<via x="24.765" y="26.67" extent="1-16" drill="0.4"/>
-<via x="26.035" y="27.94" extent="1-16" drill="0.4"/>
 <via x="23.495" y="27.94" extent="1-16" drill="0.4"/>
 <via x="23.495" y="25.4" extent="1-16" drill="0.4"/>
-<via x="26.035" y="25.4" extent="1-16" drill="0.4"/>
 <via x="26.035" y="29.845" extent="1-16" drill="0.4"/>
 <via x="23.495" y="30.48" extent="1-16" drill="0.4"/>
@@
 <via x="8.89" y="26.035" extent="1-16" drill="0.4"/>
 <via x="18.6912" y="27.94" extent="1-16" drill="0.4"/>
+<contactref element="Q3" pad="7"/>
+<contactref element="Q3" pad="8"/>
+<contactref element="Q3" pad="E1"/>
+<contactref element="Q3" pad="E2"/>
+<contactref element="Q3" pad="PAD"/>
+<wire x1="22.5" y1="23.495" x2="25.675" y2="26.67" width="1.778" layer="1"/>
+<wire x1="5.715" y1="23.495" x2="22.5" y2="23.495" width="1.778" layer="1"/>
 </signal>
 <signal name="EXT2_D">
 <contactref element="J2" pad="3"/>
 <contactref element="EXT2_L" pad="C"/>
-<contactref element="Q4" pad="EXP"/>
-<contactref element="Q4" pad="MB"/>
-<wire x1="25.585" y1="36.83" x2="22.41" y2="33.655" width="1.778" layer="1"/>
-<wire x1="22.41" y1="33.655" x2="5.715" y2="33.655" width="1.778" layer="1"/>
+<contactref element="Q4" pad="5"/>
+<contactref element="Q4" pad="6"/>
 <polygon width="0.1524" layer="16" isolate="0.4064" thermals="no">
 <vertex x="3.175" y="32.385"/>
@@
 <vertex x="27.686" y="32.385"/>
 </polygon>
-<via x="24.765" y="36.83" extent="1-16" drill="0.4"/>
-<via x="26.035" y="38.1" extent="1-16" drill="0.4"/>
 <via x="23.495" y="38.1" extent="1-16" drill="0.4"/>
 <via x="23.495" y="35.56" extent="1-16" drill="0.4"/>
-<via x="26.035" y="35.56" extent="1-16" drill="0.4"/>
 <via x="26.035" y="40.64" extent="1-16" drill="0.4"/>
 <via x="23.495" y="40.64" extent="1-16" drill="0.4"/>
@@
 <via x="8.89" y="34.29" extent="1-16" drill="0.4"/>
 <via x="8.89" y="36.83" extent="1-16" drill="0.4"/>
+<contactref element="Q4" pad="7"/>
+<contactref element="Q4" pad="8"/>
+<contactref element="Q4" pad="E1"/>
+<contactref element="Q4" pad="E2"/>
+<contactref element="Q4" pad="PAD"/>
+<wire x1="22.5" y1="33.655" x2="25.675" y2="36.83" width="1.778" layer="1"/>
+<wire x1="5.715" y1="33.655" x2="22.5" y2="33.655" width="1.778" layer="1"/>
 </signal>
 <signal name="EXT1">
@@
 <contactref element="R46" pad="2"/>
 <contactref element="Q3" pad="4"/>
-<wire x1="30.392" y1="29.083" x2="29.884" y2="28.575" width="0.3048" layer="1"/>
-<wire x1="29.884" y1="28.575" x2="28.76" y2="28.575" width="0.3048" layer="1"/>
+<wire x1="27.435" y1="27.645" x2="28.954" y2="27.645" width="0.3048" layer="1"/>
+<wire x1="28.954" y1="27.645" x2="30.392" y2="29.083" width="0.3048" layer="1"/>
 </signal>
 <signal name="EXT2_G">
 <contactref element="R47" pad="2"/>
 <contactref element="Q4" pad="4"/>
-<wire x1="30.265" y1="39.37" x2="29.63" y2="38.735" width="0.3048" layer="1"/>
-<wire x1="29.63" y1="38.735" x2="28.76" y2="38.735" width="0.3048" layer="1"/>
+<wire x1="27.435" y1="37.805" x2="28.7" y2="37.805" width="0.3048" layer="1"/>
+<wire x1="28.7" y1="37.805" x2="30.265" y2="39.37" width="0.3048" layer="1"/>
 </signal>
 <signal name="EXT_L">
