File: projects/B4SR3350/V0/B4SR3350.brd (EAGLE design)
At the start: 299.1 x 33.3 mm, 290 parts, among them IC1 A4403, IC10 TMC5130, IC12 CD4072B-TSSOP14, IC13 TMC5130, IC2 LDO-TS1117CW-3V3, IC3 ATSAM4S8C, IC4 SI87XXIS, IC5 74HC125TSSOP14, IC6 TMC5130, IC7 TMC5130, IC8 TMC5130, IC9 TMC5130, J1 ZX62-AB-5PA, J2 MOLEX-SD-47571-001, J3 MSTBV8, J4 U.FL, Q1 NX138BKS, Q2 NX138BKS, Q3 NX138BKS, Q4 AON7524, Q5 AON7524, Q6 AON7524, Q7 AON7524, U1 ESP8266, X1 12MHz, X2 KK-254-4, X3 KK-254-4, X4 KK-254-4, X5 KK-254-4, X6 KK-254-4, X7 KK-254-4, X9 KK-254-4

Commit message: 60% of layout/routing for new B4SR
Parts:
- moved IC12 338.2 mm to (-83.8, 64.8), turned to 0 degrees
- moved R26 24.7 mm to (149.9, -7.62)
- moved C112 21.5 mm to (143.5, -7.62), turned to 0 degrees
- moved R19 18.5 mm to (143.5, -3.81), turned to 0 degrees
- moved R18 18.2 mm to (138.4, -7.62), turned to 0 degrees
- moved C113 17.3 mm to (139.7, -3.81), turned to 0 degrees
- moved R25 13.0 mm to (134.6, -6.35)
- moved C117 5.00 mm to (146.6, 3.56), turned to 270 degrees
- moved C116 4.62 mm to (149.0, 7.62), turned to 0 degrees
- moved L7 3.10 mm to (148.7, 9.65), turned to 315 degrees
- moved R32 2.79 mm to (150.0, 13.0)
- moved C115 1.65 mm to (141.2, 3.56), turned to 270 degrees
- moved C114 1.06 mm to (137.0, 3.81), turned to 90 degrees
- moved R24 0.97 mm to (137.2, 8.51)
- moved X8 0.92 mm to (138.9, 6.22)
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Connections:
- net SG_TST_E1: now also IC12.10; no longer IC12.5
- net SG_TST_E2: now also IC12.11; no longer IC12.4
- net SG_TST_E3: now also IC12.12; no longer IC12.3
- net SG_TST_X: now also IC12.3; no longer IC12.12
- net SG_TST_Y: now also IC12.4; no longer IC12.11
- net SG_TST_Z: now also IC12.5; no longer IC12.10
Routing:
- net Z_DIR: track 6.85 -> 136.5 mm, vias 0 -> 1
- net Z_STEP: track 6.27 -> 135.3 mm, vias 0 -> 1
- net Z_EN: track 5.70 -> 132.4 mm, vias 0 -> 1
- net Y_DIR: track 11.2 -> 116.5 mm, vias 0 -> 1
- net X_STEP: track 128.1 -> 37.8 mm
- net MOT_MISO: track 78.3 -> 0.00 mm, vias 4 -> 0
- net MOT_MOSI: track 77.9 -> 0.00 mm, vias 4 -> 0
- net MOT_SCK: track 77.4 -> 0.00 mm, vias 4 -> 0
- net ENN: track 141.8 -> 67.5 mm, vias 3 -> 0
- net SG_TST_E1: track 76.9 -> 11.8 mm, vias 1 -> 0
- net +3V3: track 181.3 -> 129.0 mm, vias 9 -> 4
- net SG_TST_E2: track 62.5 -> 11.8 mm, vias 1 -> 0
- net GND: track 734.3 -> 692.5 mm
- net SG_TST_E3: track 39.9 -> 11.8 mm, vias 1 -> 0
- net SAM_TFR_RDY: track 27.1 -> 0.00 mm, vias 2 -> 0
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
Commit message: B4SR stuff, mostly, and APSR V5 schematic
Parts:
- removed IC4: SI87XXIS, misc:SOIC08-FAIRCHILD
- removed SJ1, SJ2: (no value), jumper:SJ
- added C118, C119, C120, C121, C38, C39: 2.2n, resistor:C0603
- added D4, D5, D6: BAT54C, diode:SOT23
- added J5: (no value), SparkFun-Connectors:1X03_SMALL
- added R79, R81, R86, R87, R88, R89, R90, R91, R92, R93, R94, R95: 10K, resistor:R0603
- RESET: value (none) -> PTS647; device misc:EVQQ2 -> misc:PTS647
- moved R65 456.2 mm to (293.2, 12.7), turned to 180 degrees
- moved C124 378.0 mm to (252.9, 10.7), turned to 180 degrees
- moved IC12 340.3 mm to (251.5, 6.73), turned to 270 degrees
- moved RESET 244.8 mm to (111.5, 3.56)
- moved R11 229.4 mm to (116.7, 31.6)
- moved USB_L 219.6 mm to (113.2, 31.6), turned to 270 degrees
- moved F1 217.3 mm to (93.9, 10.9), turned to 270 degrees
- moved R16 209.1 mm to (120.2, 5.26), turned to 90 degrees
- moved C45 193.4 mm to (135.5, 28.6), turned to 135 degrees
- moved R9 185.6 mm to (68.2, 27.7), turned to 180 degrees
- moved 5V 182.2 mm to (71.6, 27.7), turned to 90 degrees
- moved R8 180.3 mm to (68.2, 29.7), turned to 180 degrees
- moved R14 179.5 mm to (96.5, 10.7), turned to 180 degrees
- moved VIN 176.8 mm to (71.6, 30.1), turned to 90 degrees
- moved 3V3 169.4 mm to (71.6, 25.3), turned to 90 degrees
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Connections:
- net N$2 renamed E1_FUSED
- net N$5 renamed E3_FUSED
- net N$6 renamed E2_FUSED
- removed net EXT1: R50.1
- removed net EXT2: R51.1
- removed net EXT3: R52.1
- removed net ZVSEL: SJ1.2, SJ2.2, Z_STOP.2
- new net E1_STOP_IN: E1_STOP.1, R89.2, R94.1
- new net E2_STOP_IN: E2_STOP.1, R87.2, R92.1
- new net E3_STOP_IN: E3_STOP.1, R81.2, R90.1
- new net X_STOP_IN: R88.2, R93.1, X_STOP.1
- new net Y_STOP_IN: R86.2, R91.1, Y_STOP.1
- net +12V: no longer SJ2.1
- net +3V3: now also D4.3, D5.3, D6.3, R90.2, R91.2, R92.2, R93.2, R94.2, R95.2, Z_STOP.2; no longer IC4.8, SJ1.1
- net +5V: now also J5.2
- net E1_STOP: now also C121.1, D6.1, R89.1; no longer E1_STOP.1
- net E2_STOP: now also C119.1, D5.2, R87.1; no longer E2_STOP.1
- net E3_STOP: now also C39.1, D5.1, R81.1; no longer E3_STOP.1
- net ESP_EN: now also U1.7
- net FAN1: now also IC3.21; no longer IC3.18
- net FAN3: now also IC3.18; no longer IC3.21
- net GND: now also C118.2, C119.2, C120.2, C121.2, C38.2, C39.2, J5.3, RESET.B1, RESET.B2; no longer IC4.3, IC4.5, RESET.B, RESET.B'
- net HEATER1: now also R50.1
- net HEATER2: now also R51.1
- net HEATER3: now also R52.1
- net RESET: now also RESET.A2; no longer RESET.A'
- net SERVO: now also J5.1
- net SG_TST_E1: now also IC12.5; no longer IC12.10
- net SG_TST_E2: now also IC12.4; no longer IC12.11
- net SG_TST_E3: now also IC12.3; no longer IC12.12
- net SG_TST_X: now also IC12.12; no longer IC12.3
- net SG_TST_Y: now also IC12.11; no longer IC12.4
- net SG_TST_Z: now also IC12.10; no longer IC12.5
- net T_BED: now also C42.1, IC3.5, R37.1; no longer C44.1, IC3.3, R36.1
- net T_BED_IN: now also BED.2, R37.2, R41.1; no longer BED.1, R36.2, R43.1
- net T_EXT1_IN: now also EXT1.2; no longer EXT1.1
- net T_EXT2: now also C44.1, IC3.3, R36.1; no longer C42.1, IC3.5, R37.1
- net T_EXT2_IN: now also EXT2.2, R36.2, R43.1; no longer EXT2.1, R37.2, R41.1
- net T_EXT3_IN: now also EXT3.2; no longer EXT3.1
- net VSSA: now also BED.1, EXT1.1, EXT2.1, EXT3.1; no longer BED.2, EXT1.2, EXT2.2, EXT3.2
- net X_DIR: now also IC3.38; no longer IC3.49
- net X_STOP: now also C120.1, D6.2, R88.1; no longer X_STOP.1
- net Y_DIR: now also IC3.49; no longer IC3.38
- net Y_STOP: now also C118.1, D4.2, R86.1; no longer Y_STOP.1
- net Z_STOP: now also C38.1, D4.1, R79.1; no longer IC4.6
- net Z_STOP_IN: now also R79.2, R95.1; no longer IC4.2
Routing:
- net GND: track 692.5 -> 1429.2 mm, vias 139 -> 263
- net +3V3: track 129.0 -> 550.3 mm, vias 4 -> 40
- net ENN: track 67.5 -> 342.2 mm, vias 0 -> 12
- net +12V: track 331.2 -> 575.8 mm, vias 1 -> 13
- net MOT_SCK: track 0.00 -> 216.0 mm, vias 0 -> 9
- net MOT_MOSI: track 0.00 -> 211.6 mm, vias 0 -> 9
- net MOT_MISO: track 0.00 -> 208.6 mm, vias 0 -> 9
- net Y_STEP: track 0.00 -> 157.9 mm, vias 0 -> 4
- net Y_EN: track 0.00 -> 152.8 mm, vias 0 -> 4
- net SG_TST: track 0.00 -> 148.6 mm, vias 0 -> 2
- net X_DIR: track 0.00 -> 136.6 mm, vias 0 -> 2
- net PWR_FAIL_DET2: track 0.00 -> 93.7 mm, vias 0 -> 2
- net BED: track 0.00 -> 92.3 mm, vias 0 -> 1
- net X_STEP: track 37.8 -> 129.6 mm
- net HEATER1: track 0.00 -> 90.4 mm, vias 0 -> 1
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- added copper zone on layer 1, net +3V3
- added copper zone on layer 16, net +3V3
- added copper zone on layer 1, net +5V
- added copper zone on layer 16, net A1_Z
- added copper zone on layer 16, net A2_Z
- added copper zone on layer 16, net B1_Z
- added copper zone on layer 16, net B2_Z
- added copper zone on layer 1, net BED_D
- added copper zone on layer 16, net BED_D
- added copper zone on layer 1, net EXT1_D
- added copper zone on layer 16, net EXT1_D
- added copper zone on layer 1, net EXT2_D
- added copper zone on layer 16, net EXT2_D
- added copper zone on layer 1, net EXT3_D
- added copper zone on layer 1, net LX
- added copper zone on layer 1, net VOUT
