File: projects/B4SR3350/V0/B4SR3350.sch (EAGLE design)
At the start: 272 parts, among them IC1 A4403, IC10 TMC21X0-LA, IC11 TMC21X0-LA, IC13 TMC21X0-LA, IC14 CD4072B, IC2 LDO-TS1117CW-3V3, IC3 ATSAM4S8C, IC4 SI87XXIS, IC5 74HC125, IC6 74S08D, IC7 TMC21X0-LA, IC8 TMC21X0-LA, IC9 TMC21X0-LA, J1 MOLEX-105162-001, J2 MSTBV6, J3 ZX62-AB-5PA, Q1 NX138BKS, Q2 NX138BKS, Q3 BUK9Y53-100B, Q4 BUK9Y53-100B, Q5 BUK9Y53-100B, X1 KK-254-4, X2 12MHz, X3 KK-254-2, X4 KK-254-4, X5 KK-254-4, X6 KK-254-4, X7 KK-254-4, X8 KK-254-4, X9 KK-254-4

Commit message: 60% of layout/routing for new B4SR
Parts:
- removed C118, C120: 100n, resistor:C-EUC0603
- removed C119: 22n, resistor:C-EUC0603
- removed C121: 100u, resistor:CPOL-USD
- removed C122, C123: 470p, resistor:C-EUC0402
- removed C38, C39: 10u, resistor:C-EUC0603
- removed ESP8266: (no value), adafruit:ESP-12
- removed EXP_1, EXP_2: 057-010-1, con-panduit:057-010-1
- removed IC11: TMC21X0-LA, SilentStepStick-TMC2130_v11:TMC21X0-LA
- removed IC14: CD4072B, misc:CD4072B
- removed L6: 4n7H, Zero_V1.0:INDUCTOR-0603
- added BED_L: (no value), led:LEDCHIPLED_0805
- added C126: 4u7, resistor:C-EUC0603
- added C127: 470n, resistor:C-EUC0603
- added C128, C129, C130, C132: 100n, resistor:C-EUC0603
- added C131: 22n, resistor:C-EUC0603
- added C133: 100u, resistor:CPOL-USD
- added C134, C135, C136, C137: 470p, resistor:C-EUC0402
- added E1_STOP, E2_STOP, E3_STOP: KK-254-3, con-other:KK-254-3
- added FAN5, FAN6: KK-254-2, con-other:KK-254-2
- added IC12: CD4072B-TSSOP14, misc:CD4072B-TSSOP14
- added J4: U.FL, misc:U.FL
- added L7: 4.3nH, Zero_V1.0:INDUCTOR-0402
- added L8: 2.2nH, Zero_V1.0:INDUCTOR-0402
- added PANEL: 057-010-1, con-panduit:057-010-1
- added Q6, Q7: AON7524, misc:AON7524
- added R80: 200R, resistor:R-US_R0603
- added R82, R83: 0R11, resistor:R-US_R1206
- added R84: 20K, resistor:R-TRIMM3103
- added R85: 20K, resistor:R-US_R0603
- added U1: ESP8266, SparkFun-RF:ESP8266
- added U2: (no value), misc:W25QXX
- C100, C48, C61, C74, C87: value 4u7 -> 470n
- C103, C51, C64, C77, C90: value 22n -> 100n
- C104, C52, C65, C78, C91: value 100u -> 22n; device resistor:CPOL-USD -> resistor:C-EUC0603
- C106, C54, C67, C80, C93: value 100n -> 100u; device resistor:C-EUC0603 -> resistor:CPOL-USD
- C111: value 100n -> 1u; device rcl:C-EUC0603 -> resistor:C-EUC0603
- C112: value 2.2u -> 100n
- C113: value 100n -> 10u
- C114: value 4u7 -> 6.8p
- C115: value 470n -> 6.8p
- C116: value 100n -> 3.0p
- C117: value 100n -> 2.4p
- C124: value 470p -> 100n; device resistor:C-EUC0402 -> rcl:C-EUC0603
- C125: value 470p -> 100n; device resistor:C-EUC0402 -> resistor:C-EUC0603
- C45: value 100n -> 2.2u
- C47, C60, C73, C86, C99: value 470n -> 4u7
- ERASE: device jumper:JP1Q -> SparkFun-Connectors:CONN_02SMALL
- IC10, IC13, IC7, IC8, IC9: value TMC21X0-LA -> TMC5130; device SilentStepStick-TMC2130_v11:TMC21X0-LA -> TMC5130_3D_Printer_BOARD_V_2:TMC5130
- IC5: value 74HC125 -> 74HC125TSSOP14; device misc:74HC125 -> misc:74HC125TSSOP14
- IC6: value 74S08D -> TMC5130; device 74xx-us:74S08D -> TMC5130_3D_Printer_BOARD_V_2:TMC5130
- J1: value MOLEX-105162-001 -> ZX62-AB-5PA; device misc:MOLEX-105162-001 -> Arduino:ZX62-AB-5PA
- J2: value MSTBV6 -> MOLEX-SD-47571-001; device con-phoenix-508:MSTBV6 -> misc:MOLEX-SD-47571-001
- J3: value ZX62-AB-5PA -> MSTBV8; device Arduino:ZX62-AB-5PA -> con-phoenix-508:MSTBV8
- Q3: value BUK9Y53-100B -> NX138BKS; device misc:BUK9Y53-100B -> misc:NX138BKS
- Q4, Q5: value BUK9Y53-100B -> AON7524; device misc:BUK9Y53-100B -> misc:AON7524
- R24: value 470R -> 1k
- R39: value 4K7 0.1% -> 10K
- R42, R43: value 1K -> 4K7 0.1%
- R46, R47: value 180R -> 1K
- R48, R49: value 4K7 -> 1K
- R51, R52: value 0R11 -> 180R; device resistor:R-US_R1206 -> resistor:R-US_R0603
- R53: value 20K -> 180R; device resistor:R-TRIMM3103 -> resistor:R-US_R0603
- R54: value 20K -> 4K7
- R55, R56: value 0R11 -> 4K7; device resistor:R-US_R1206 -> resistor:R-US_R0603
- R57: value 20K -> 4K7; device resistor:R-TRIMM3103 -> resistor:R-US_R0603
- R58, R62, R66, R70: value 20K -> 0R11; device resistor:R-US_R0603 -> resistor:R-US_R1206
- R60, R64, R68, R76: value 0R11 -> 20K; device resistor:R-US_R1206 -> resistor:R-TRIMM3103
- R61, R65, R69, R77: device resistor:R-TRIMM3103 -> resistor:R-US_R0603
- R71: value 4K7 0.1% -> 0R11; device resistor:R-US_R0603 -> resistor:R-US_R1206
- R72: value 10K -> 20K; device resistor:R-US_R0603 -> resistor:R-TRIMM3103
- R73: value 180R -> 20K
- R74: value 4K7 -> 0R11; device resistor:R-US_R0603 -> resistor:R-US_R1206
- R78: value 20K -> 12K 1%
- X1: value KK-254-4 -> 12MHz; device con-other:KK-254-4 -> misc:CRYSTAL-4PIN5X3
- X2: value 12MHz -> KK-254-4; device misc:CRYSTAL-4PIN -> con-other:KK-254-4
- X3: value KK-254-2 -> KK-254-4; device con-other:KK-254-2 -> con-other:KK-254-4
- X8: value KK-254-4 -> (none); device con-other:KK-254-4 -> misc:CRYSTAL-4PIN3X2
- renumbered EXT2_L1 to EXT3_L
Connections:
- net FAN_E2 renamed HEATER2
- removed net AMID_Z: X6-1.S, X7-2.S
- removed net BED_L1: EXT3_L.A, R74.1
- removed net BED_OUT: R50.2, X3-1.S
- removed net BMID_Z: X6-4.S, X7-3.S
- removed net E1_FUSED: F2.2, J2-5.1
- removed net E2_FUSED: F3.2, J2-3.1
- removed net ESP_RXD: ESP8266.TXD, R23.2
- removed net ESP_TXD: ESP8266.RXD, R24.2
- removed net ESP_VIN: ESP8266.VCC, L6.2
- removed net EXT2_D1: EXT3_L.C, J2-2.1, Q5.D
- removed net EXT2_G1: Q5.G, R73.2
- removed net EXT_L: EXT1_L.A, R48.1
- removed net FAN_E1: IC3.PC3
- removed net FAN_MOBO: IC3.PA18/PGMD6/AD1
- removed net FAN_PART: IC3.PC13/AD10
- removed net LCD_BEEP: EXP_2-1.S, IC3.PB13/DAC0, IC3.PC18, IC3.PC23, IC3.PC24, IC3.PC25, IC3.TDO/TRACESWO/PB5, IC3.TMS/SWDIO/PB6
- removed net LCD_CS: IC3.PC19, IC6A.I1, IC6B.I0, IC6B.I1, IC6D.I1
- removed net LCD_CS_BUF: EXP_2-4.S, IC6B.O
- removed net LCD_ENC_A: EXP_1-5.S, IC3.TCK/SWCLK/PB7
- removed net LCD_ENC_B: EXP_1-3.S, IC3.PC20
- removed net N$1: EXT3-1.S, R71.1, R72.2
- removed net N$3: F4.2, J2-1.1
- removed net SD_MOSI_BUF: EXP_1-6.S, IC5A.O
- removed net SD_SCK_BUF: EXP_1-2.S, IC5B.O
- removed net T_EXT_IN: EXT1-1.S, R37.2, R40.1
- removed net T_EXT_IN1: EXT2-1.S, R38.2, R39.1
- new net ANTENNA: C117.1, J4.SIGNAL, L8.2
- new net A_Z2: X3-1.S, X7-2.S
- new net BED_D: BED_L.C, J3-8.1, Q7.D
- new net BED_G: Q7.G, R53.2
- new net B_Z2: X3-4.S, X7-3.S
- new net E1_STOP: E1_STOP-1.S, IC3.PC31
- new net E2_STOP: E2_STOP-1.S, IC3.PC25
- new net E3_STOP: E3_STOP-1.S, IC3.PC24
- new net ESP_XIN: C115.1, U1.XTAL_IN, X8.1
- new net ESP_XOUT: C114.2, U1.XTAL_OUT, X8.3
- new net EXT1_L: EXT1_L.A, R54.1
- new net EXT2_L: EXT2_L.A, R55.1
- new net EXT3: R52.1
- new net EXT3_D: EXT3_L.C, J3-6.1, Q6.D
- new net EXT3_G: Q6.G, R52.2
- new net EXT3_L: EXT3_L.A, R56.1
- new net FAN1: IC3.PA19/PGMD7/AD2, R44.1
- new net FAN1_G1: Q1A.G, R44.2
- new net FAN2: IC3.PC15/AD11, R45.1
- new net FAN2_G1: Q1B.G, R45.2
- new net FAN5_D: FAN5-2.S, Q3A.D
- new net FAN6_D: FAN6-2.S, Q3B.D
- new net FLASH_CLK: R80.2, U2.CLK
- new net FLASH_CS: U1.SPICS0/SD_CMD, U2./CS
- new net FLASH_D: U1.SPID/SD_DATA_1, U2.DI
- new net FLASH_HOLD: U1.SPIHD/SD_DATA_2, U2./HOLD
- new net FLASH_Q: U1.SPIQ/SD_DATA_0, U2.DO
- new net FLASH_WP: U1.SPIWP/SD_DATA_3, U2./WP
- new net HEATER1: IC3.PA16/PGMD4
- new net HEATER3: IC3.PA20/PGMD8/AD3
- new net LNA: C116.1, L8.1, U1.LNA
- new net N$5: F4.2, J3-5.1
- new net N$6: F3.2, J3-3.1
- new net RES12K: R78.2, U1.RES12K
- new net SERVO: IC3.PC26
- new net SPICLK: R80.1, U1.SPICLK/SD_CLK
- new net T_EXT1_IN: EXT1-1.S, R38.2, R42.1
- new net T_EXT2_IN: EXT2-1.S, R37.2, R41.1
- new net T_EXT3_IN: EXT3-1.S, R39.2, R40.1
- new net URXD: R23.2, U1.U0RXD
- new net URXD1: IC3.PB2/AD6, PANEL-9.S
- new net UTXD: R24.2, U1.U0TXD
- new net UTXD1: IC3.PB3/AD7, PANEL-10.S
- new net VDD3P3: L7.2, U1.VDD3P3@3, U1.VDD3P3@4
- net +12V: now also C103.1, C106.+, C128.2, C129.1, C130.1, C132.1, C133.+, C51.1, C54.+, C64.1, C67.+, C77.1, C80.+, C90.1, C93.+, FAN5-1.S, FAN6-1.S, IC6.VS, IC6.VSA, J3-7.1, R54.2, R55.2, R56.2, R57.2; no longer C104.+, C106.1, C116.2, C117.1, C118.1, C120.1, C121.+, C52.+, C54.1, C65.+, C67.1, C78.+, C80.1, C91.+, C93.1, IC11.VS, IC11.VSA, R48.2, R49.2, R74.2
- net +3V3: now also C112.1, C124.1, C125.1, C45.1, E1_STOP-2.S, E2_STOP-2.S, E3_STOP-2.S, IC12-P.VCC, IC6.VCC_IO, J2.VDD, L7.1, PANEL-8.S, U1.VDDA@1, U1.VDDA@30, U1.VDDD, U1.VDDPST@11, U1.VDDPST@17, U2.VCC; no longer C38.1, C39.1, C44.1, IC11.VCC_IO, IC14-P.VCC, J1.VDD, L6.1
- net +5V: now also C100.1, C127.1, C48.1, C61.1, C74.1, C87.1, IC6.VCC, PANEL-1.S, R61.2, R65.2, R69.2, R73.2, R77.2, R85.2; no longer C115.1, C45.1, C47.1, C60.1, C73.1, C86.1, C99.1, EXP_2-10.S, IC11.VCC, IC6P.VCC, R54.2, R58.2, R62.2, R66.2, R70.2, R78.2
- net 5V_E1: now also C126.1, IC13.5VOUT; no longer C87.1, IC10.5VOUT
- net 5V_E2: now also C47.1, IC6.5VOUT; no longer C100.1, IC11.5VOUT
- net 5V_E3: now also C73.1, IC8.5VOUT; no longer C114.1, IC13.5VOUT
- net 5V_X: now also C86.1, IC9.5VOUT; no longer C48.1, IC7.5VOUT
- net 5V_Y: now also C99.1, IC10.5VOUT; no longer C61.1, IC8.5VOUT
- net 5V_Z: now also C60.1, IC7.5VOUT; no longer C74.1, IC9.5VOUT
- net A1_E1: now also C134.1, IC13.OA1, X9-1.S; no longer C94.1, IC10.OA1, X8-1.S
- net A1_E2: now also C55.1, IC6.OA1, X2-1.S; no longer C107.1, IC11.OA1, X9-1.S
- net A1_E3: now also C81.1, IC8.OA1, X4-1.S; no longer C122.1, IC13.OA1, X1-1.S
- net A1_X: now also C94.1, IC9.OA1, X5-1.S; no longer C55.1, IC7.OA1, X4-1.S
- net A1_Y: now also C107.1, IC10.OA1, X6-1.S; no longer C68.1, IC8.OA1, X5-1.S
- net A1_Z: now also C68.1, IC7.OA1; no longer C81.1, IC9.OA1
- net A2_E1: now also C135.1, IC13.OA2, X9-2.S; no longer C95.1, IC10.OA2, X8-2.S
- net A2_E2: now also C56.1, IC6.OA2, X2-2.S; no longer C108.1, IC11.OA2, X9-2.S
- net A2_E3: now also C82.1, IC8.OA2, X4-2.S; no longer C123.1, IC13.OA2, X1-2.S
- net A2_X: now also C95.1, IC9.OA2, X5-2.S; no longer C56.1, IC7.OA2, X4-2.S
- net A2_Y: now also C108.1, IC10.OA2, X6-2.S; no longer C69.1, IC8.OA2, X5-2.S
- net A2_Z: now also C69.1, IC7.OA2, X3-2.S; no longer C82.1, IC9.OA2, X6-2.S
- net ADVREF: now also R42.2, R43.2; no longer R39.2, R71.2
- net B1_E1: now also C136.1, IC13.OB1, X9-4.S; no longer C96.1, IC10.OB1, X8-3.S
- net B1_E2: now also C57.1, IC6.OB1, X2-4.S; no longer C109.1, IC11.OB1, X9-3.S
- net B1_E3: now also C83.1, IC8.OB1, X4-4.S; no longer C124.1, IC13.OB1, X1-3.S
- net B1_X: now also C96.1, IC9.OB1, X5-4.S; no longer C57.1, IC7.OB1, X4-3.S
- net B1_Y: now also C109.1, IC10.OB1, X6-4.S; no longer C70.1, IC8.OB1, X5-3.S
- net B1_Z: now also C70.1, IC7.OB1, X3-3.S; no longer C83.1, IC9.OB1, X6-3.S
- net B2_E1: now also C137.1, IC13.OB2, X9-3.S; no longer C97.1, IC10.OB2, X8-4.S
- net B2_E2: now also C58.1, IC6.OB2, X2-3.S; no longer C110.1, IC11.OB2, X9-4.S
- net B2_E3: now also C84.1, IC8.OB2, X4-3.S; no longer C125.1, IC13.OB2, X1-4.S
- net B2_X: now also C97.1, IC9.OB2, X5-3.S; no longer C58.1, IC7.OB2, X4-4.S
- net B2_Y: now also C110.1, IC10.OB2, X6-3.S; no longer C71.1, IC8.OB2, X5-4.S
- net B2_Z: now also C71.1, IC7.OB2; no longer C84.1, IC9.OB2
- net BED: now also IC3.PA15/PGMD3, R53.1; no longer IC3.PC22, R50.1
- net BED_L: now also BED_L.A, R57.1; no longer EXT2_L.A, R49.1
- net BRA_E1: now also IC13.BRA, R82.1; no longer IC10.BRA, R63.1
- net BRA_E2: now also IC6.BRA, R58.1; no longer IC11.BRA, R67.1
- net BRA_E3: now also IC8.BRA, R66.1; no longer IC13.BRA, R75.1
- net BRA_X: now also IC9.BRA, R70.1; no longer IC7.BRA, R51.1
- net BRA_Y: now also IC10.BRA, R74.1; no longer IC8.BRA, R55.1
- net BRA_Z: now also IC7.BRA, R62.1; no longer IC9.BRA, R59.1
- net BRB_E1: now also IC13.BRB, R83.1; no longer IC10.BRB, R64.1
- net BRB_E2: now also IC6.BRB, R59.1; no longer IC11.BRB, R68.1
- net BRB_E3: now also IC8.BRB, R67.1; no longer IC13.BRB, R76.1
- net BRB_X: now also IC9.BRB, R71.1; no longer IC7.BRB, R52.1
- net BRB_Y: now also IC10.BRB, R75.1; no longer IC8.BRB, R56.1
- net BRB_Z: now also IC7.BRB, R63.1; no longer IC9.BRB, R60.1
- net CLK: now also J2.CLK; no longer J1.CLK
- net CMD: now also J2.CMD; no longer J1.CMD
- net CPI_E1: now also C131.1, IC13.CPI; no longer C90.1, IC10.CPI
- net CPI_E2: now also C52.1, IC6.CPI; no longer C103.1, IC11.CPI
- net CPI_E3: now also C78.1, IC8.CPI; no longer C119.1, IC13.CPI
- net CPI_X: now also C91.1, IC9.CPI; no longer C51.1, IC7.CPI
- net CPI_Y: now also C104.1, IC10.CPI; no longer C64.1, IC8.CPI
- net CPI_Z: now also C65.1, IC7.CPI; no longer C77.1, IC9.CPI
- net CPO_E1: now also C131.2, IC13.CPO; no longer C90.2, IC10.CPO
- net CPO_E2: now also C52.2, IC6.CPO; no longer C103.2, IC11.CPO
- net CPO_E3: now also C78.2, IC8.CPO; no longer C119.2, IC13.CPO
- net CPO_X: now also C91.2, IC9.CPO; no longer C51.2, IC7.CPO
- net CPO_Y: now also C104.2, IC10.CPO; no longer C64.2, IC8.CPO
- net CPO_Z: now also C65.2, IC7.CPO; no longer C77.2, IC9.CPO
- net DAT0: now also J2.DAT0; no longer J1.DAT0
- net DAT1: now also J2.DAT1; no longer J1.DAT1
- net DAT2: now also J2.DAT2; no longer J1.DAT2
- net DAT3: now also J2.DAT3; no longer J1.DAT3
- net DET: now also J2.CARD_DETECT; no longer J1.CARD_DETECT
- net E1_DIR: now also IC13.REFR_DIR, IC3.PC17; no longer IC10.REFR_DIR, IC3.TDI/PB4
- net E1_EN: now also IC13.CSN_CFG3, IC3.TMS/SWDIO/PB6; no longer IC10.CSN_CFG3, IC3.PA4/PGMNCMD
- net E1_STEP: now also IC13.REFL_STEP, IC3.PC18; no longer IC10.REFL_STEP, IC3.PC28
- net E2_DIR: now also IC3.PA1/PGMEN1, IC6.REFR_DIR; no longer IC11.REFR_DIR, IC3.PC9
- net E2_EN: now also IC3.PA0/PGMEN0, IC6.CSN_CFG3; no longer IC11.CSN_CFG3, IC3.PA3
- net E2_STEP: now also IC3.PC16, IC6.REFL_STEP; no longer IC11.REFL_STEP, IC3.PC10
- net E3_DIR: now also IC3.PC9, IC8.REFR_DIR; no longer IC13.REFR_DIR
- net E3_EN: now also IC3.PA3, IC8.CSN_CFG3; no longer IC13.CSN_CFG3
- net E3_STEP: now also IC3.PC10, IC8.REFL_STEP; no longer IC13.REFL_STEP
- net EDR_CONN: now also U1.SPICS2/GPIO0; no longer ESP8266.GPIO0
- net ENN: now also IC6.DRV_ENN_CFG6; no longer IC11.DRV_ENN_CFG6
- net ESP_CS: now also U1.MTDO/SPICS/GPIO15; no longer ESP8266.GPIO15
- net ESP_DATA_RDY: now also IC3.PC3; no longer IC3.PC26
- net ESP_EN: no longer ESP8266.CH_PD
- net ESP_RST: now also U1.EXT_RSTB; no longer ESP8266.RESET
- net EXT1: now also R50.1; no longer IC3.PA20/PGMD8/AD3, R46.1
- net EXT1_D: now also J3-2.1, Q4.D; no longer J2-6.1, Q3.D
- net EXT1_G: now also Q4.G, R50.2; no longer Q3.G, R46.2
- net EXT2: now also R51.1; no longer IC3.PC15/AD11, R47.1, R73.1
- net EXT2_D: now also J3-4.1, Q5.D; no longer J2-4.1, Q4.D
- net EXT2_G: now also Q5.G, R51.2; no longer Q4.G, R47.2
- net FAN1_G: now also Q2A.G, R46.2; no longer Q1A.G, R42.2
- net FAN2_G: now also Q2B.G, R47.2; no longer Q1B.G, R43.2
- net FAN3: now also IC3.PC13/AD10, R46.1; no longer R42.1
- net FAN3_G: now also Q3A.G, R48.2; no longer Q2A.G, R44.2
- net FAN4: now also IC3.TDO/TRACESWO/PB5, R47.1; no longer R43.1
- net FAN4_G: now also Q3B.G, R49.2; no longer Q2B.G, R45.2
- net FAN5: now also IC3.PC22, R48.1; no longer R44.1
- net FAN6: now also IC3.PB13/DAC0, R49.1; no longer R45.1
- net GND: now also C102.2, C103.2, C106.-, C114.1, C116.2, C126.2, C127.2, C128.1, C129.2, C130.2, C133.-, C134.2, C135.2, C136.2, C137.2, C50.2, C51.2, C54.-, C63.2, C64.2, C67.-, C76.2, C77.2, C80.-, C89.2, C90.2, C93.-, E1_STOP-3.S, E2_STOP-3.S, E3_STOP-3.S, IC10.GNDP, IC10.GND_PAD, IC12-2.I0, IC12-P.GND, IC13.GNDP, IC13.GND_PAD, IC6.CLK, IC6.ENCB_DCEN_CFG4, IC6.GND, IC6.GNDA, IC6.GNDP, IC6.GND_PAD, IC6.TST_MODE, IC7.GNDP, IC7.GND_PAD, IC8.GNDP, IC8.GND_PAD, IC9.GNDP, IC9.GND_PAD, J2.GND, J2.VSS, J4.GND, PANEL-2.S, Q1A.S, Q1B.S, Q2A.S, Q2B.S, Q3A.S, Q3B.S, Q4.S, Q5.S, Q6.S, Q7.S, R58.2, R60.A, R62.2, R64.A, R66.2, R68.A, R70.2, R71.2, R72.A, R74.2, R76.A, R78.1, R82.2, R83.2, R84.A, U1.GND, U2.GND, X1.2, X1.4, X8.2, X8.4; no longer C104.-, C105.2, C106.2, C114.2, C116.1, C118.2, C121.-, C122.2, C123.2, C38.2, C39.2, C52.-, C53.2, C54.2, C65.-, C66.2, C67.2, C78.-, C79.2, C80.2, C91.-, C92.2, C93.2, ESP8266.GND, EXP_1-9.S, EXP_2-9.S, IC11.CLK, IC11.ENCB_DCEN_CFG4, IC11.GND, IC11.GNDA, IC11.TST_MODE, IC14-2.I0, IC14-P.GND, IC6C.I0, IC6C.I1, IC6P.GND, J1.VSS, J3.GND, R51.2, R52.2, R53.E, R55.2, R56.2, R57.E, R60.2, R61.E, R64.2, R65.E, R68.2, R69.E, R76.2, R77.E, X2.2, X2.4, X3-2.S
- net IREF_E1: now also IC13.AIN_IREF, R84.S; no longer IC10.AIN_IREF, R65.S
- net IREF_E2: now also IC6.AIN_IREF, R60.S; no longer IC11.AIN_IREF, R69.S
- net IREF_E3: now also IC8.AIN_IREF, R68.S; no longer IC13.AIN_IREF, R77.S
- net IREF_X: now also IC9.AIN_IREF, R72.S; no longer IC7.AIN_IREF, R53.S
- net IREF_Y: now also IC10.AIN_IREF, R76.S; no longer IC8.AIN_IREF, R57.S
- net IREF_Z: now also IC7.AIN_IREF, R64.S; no longer IC9.AIN_IREF, R61.S
- net LCD_ENC_SW: now also IC3.PC20, PANEL-7.S; no longer EXP_2-2.S, IC3.PC21
- net LCD_MISO_BUF: now also PANEL-6.S; no longer EXP_1-1.S
- net LCD_MOSI: no longer IC6A.I0
- net LCD_MOSI_BUF: now also IC5A.O, PANEL-5.S; no longer EXP_2-3.S, IC6A.O
- net LCD_SCK: no longer IC6D.I0
- net LCD_SCK_BUF: now also IC5B.O, PANEL-4.S; no longer EXP_2-5.S, IC6D.O
- net LCD_SD_CS: now also IC3.PC19, PANEL-3.S; no longer EXP_1-4.S, IC3.PB14/DAC1
- net MISO: now also U1.MTDI/SPIQ/GPIO12; no longer ESP8266.GPIO12
- net MOSI: now also U1.MTCK/SPID/GPIO13; no longer ESP8266.GPIO13
- net MOT_MISO: now also IC6.SDO_NAO_CFG0; no longer IC11.SDO_NAO_CFG0
- net MOT_MOSI: now also IC6.SDI_NAI_CFG1; no longer IC11.SDI_NAI_CFG1
- net MOT_SCK: now also IC6.SCK_CFG2; no longer IC11.SCK_CFG2
- net N$2: now also F2.2, J3-1.1; no longer Q1A.S, Q1B.S, Q2A.S, Q2B.S, Q3.S, Q4.S, Q5.S
- net N$4: now also IC12-1.I0, IC12-2.O; no longer IC14-1.I0, IC14-2.O
- net PWR_FAIL_DET2: now also IC3.PC12/AD12; no longer IC3.PC30/AD14
- net REFIN_E1: now also R84.E, R85.1; no longer R65.A, R66.1
- net REFIN_E2: now also R60.E, R61.1; no longer R69.A, R70.1
- net REFIN_E3: now also R68.E, R69.1; no longer R77.A, R78.1
- net REFIN_X: now also R72.E, R73.1; no longer R53.A, R54.1
- net REFIN_Y: now also R76.E, R77.1; no longer R57.A, R58.1
- net REFIN_Z: now also R64.E, R65.1; no longer R61.A, R62.1
- net SAM_TFR_RDY: now also IC3.PC7, U1.GPIO4; no longer ESP8266.GPIO4, IC3.PA7/XIN32/PGMNVALID
- net SG_TST: now also IC12-1.O, IC3.PC27; no longer IC14-1.O, IC3.PA1/PGMEN1
- net SG_TST_E1: now also IC12-2.I1, IC13.SWP_DIAG1; no longer IC10.SWP_DIAG1, IC14-2.I1
- net SG_TST_E2: now also IC12-2.I2, IC6.SWP_DIAG1; no longer IC11.SWP_DIAG1, IC14-2.I2
- net SG_TST_E3: now also IC12-2.I3, IC8.SWP_DIAG1; no longer IC13.SWP_DIAG1, IC14-2.I3
- net SG_TST_X: now also IC12-1.I1, IC9.SWP_DIAG1; no longer IC14-1.I1, IC7.SWP_DIAG1
- net SG_TST_Y: now also IC10.SWP_DIAG1, IC12-1.I2; no longer IC14-1.I2, IC8.SWP_DIAG1
- net SG_TST_Z: now also IC12-1.I3, IC7.SWP_DIAG1; no longer IC14-1.I3, IC9.SWP_DIAG1
- net SPCK: now also U1.MTMS/SPICLK/GPIO14; no longer ESP8266.GPIO14
- net T_BED: now also C44.1, IC3.PB0/AD4; no longer C43.1, IC3.PB1/AD5
- net T_BED_IN: now also R43.1; no longer R41.1
- net T_EXT1: now also C43.1, IC3.PC29/AD13, R38.1; no longer C42.1, IC3.PB0/AD4, IC3.PB2/AD6, IC3.PB3/AD7, IC3.PC12/AD12, IC3.PC27, IC3.PC31, R37.1
- net T_EXT2: now also C42.1, IC3.PB1/AD5, R37.1; no longer C41.1, IC3.PC29/AD13, R38.1
- net T_EXT3: now also C41.1, IC3.PC30/AD14, R39.1; no longer C112.1, R72.1
- net USB_N: now also J1.D-; no longer J3.D-
- net USB_P: now also J1.D+; no longer J3.D+
- net VBUS: now also J1.VUSB; no longer J3.VUSB
- net VCP_E1: now also C132.2, IC13.VCP; no longer C89.2, IC10.VCP
- net VCP_E2: now also C53.2, IC6.VCP; no longer C102.2, IC11.VCP
- net VCP_E3: now also C79.2, IC8.VCP; no longer C120.2, IC13.VCP
- net VCP_X: now also C92.2, IC9.VCP; no longer C50.2, IC7.VCP
- net VCP_Y: now also C105.2, IC10.VCP; no longer C63.2, IC8.VCP
- net VCP_Z: now also C66.2, IC7.VCP; no longer C76.2, IC9.VCP
- net VSSA_MON: now also IC3.PA18/PGMD6/AD1; no longer IC3.PA19/PGMD7/AD2
- net XIN: now also X1.3; no longer X2.3
- net XOUT: now also X1.1; no longer X2.1
- net X_DIR: now also IC3.PA7/XIN32/PGMNVALID, IC9.REFR_DIR; no longer IC3.PA16/PGMD4, IC7.REFR_DIR
- net X_EN: now also IC3.PA4/PGMNCMD, IC9.CSN_CFG3; no longer IC3.PA15/PGMD3, IC7.CSN_CFG3
- net X_STEP: now also IC3.PC28, IC9.REFL_STEP; no longer IC3.PC7, IC7.REFL_STEP
- net X_STOP: now also IC3.PC23; no longer IC3.PC16
- net Y_DIR: now also IC10.REFR_DIR, IC3.PA25/PGMD13; no longer IC3.PA24/PGMD12, IC8.REFR_DIR
- net Y_EN: now also IC10.CSN_CFG3, IC3.PA8/XOUT32/PGMM0; no longer IC3.PC4, IC8.CSN_CFG3
- net Y_STEP: now also IC10.REFL_STEP, IC3.PC1; no longer IC3.PC5, IC8.REFL_STEP
- net Y_STOP: now also IC3.PC21; no longer IC3.PA0/PGMEN0
- net Z_DIR: now also IC3.PA24/PGMD12, IC7.REFR_DIR; no longer IC3.PA25/PGMD13, IC9.REFR_DIR
- net Z_EN: now also IC3.PC4, IC7.CSN_CFG3; no longer IC3.PA8/XOUT32/PGMM0, IC9.CSN_CFG3
- net Z_STEP: now also IC3.PC5, IC7.REFL_STEP; no longer IC3.PC1, IC9.REFL_STEP
- net Z_STOP: now also IC3.TCK/SWCLK/PB7; no longer IC3.PC17
Other:
- moved on the sheet: C100, C101, C102, C103, C105, C107, C108, C109, C110, C111, C112, C113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

Commit message: B4SR stuff, mostly, and APSR V5 schematic
Parts:
- removed IC4: SI87XXIS, misc:SI87XXIS
- removed SJ1, SJ2: (no value), jumper:SJ
- added C118, C119, C120, C121, C38, C39: 2.2n, resistor:C-EUC0603
- added D4, D5, D6: BAT54C, diode:BAT54C
- added J5: (no value), SparkFun-Connectors:CONN_03SMALL
- added R79, R81, R86, R87, R88, R89, R90, R91, R92, R93, R94, R95: 10K, resistor:R-US_R0603
- RESET: value (none) -> PTS647; device misc:EVQQ2 -> misc:PTS647
Connections:
- net N$2 renamed E1_FUSED
- net N$5 renamed E3_FUSED
- net N$6 renamed E2_FUSED
- removed net EXT1: R50.1
- removed net EXT2: R51.1
- removed net EXT3: R52.1
- removed net ZVSEL: SJ1.2, SJ2.2, Z_STOP-2.S
- new net E1_STOP_IN: E1_STOP-1.S, R89.2, R94.1
- new net E2_STOP_IN: E2_STOP-1.S, R87.2, R92.1
- new net E3_STOP_IN: E3_STOP-1.S, R81.2, R90.1
- new net X_STOP_IN: R88.2, R93.1, X_STOP-1.S
- new net Y_STOP_IN: R86.2, R91.1, Y_STOP-1.S
- net +12V: no longer SJ2.1
- net +3V3: now also D4.CC, D5.CC, D6.CC, R90.2, R91.2, R92.2, R93.2, R94.2, R95.2, Z_STOP-2.S; no longer IC4.VDD, SJ1.1
- net +5V: now also J5.2
- net E1_STOP: now also C121.1, D6.A1, R89.1; no longer E1_STOP-1.S
- net E2_STOP: now also C119.1, D5.A2, R87.1; no longer E2_STOP-1.S
- net E3_STOP: now also C39.1, D5.A1, R81.1; no longer E3_STOP-1.S
- net ESP_EN: now also U1.CHIP_EN
- net FAN1: now also IC3.PC13/AD10; no longer IC3.PA19/PGMD7/AD2
- net FAN3: now also IC3.PA19/PGMD7/AD2; no longer IC3.PC13/AD10
- net GND: now also C118.2, C119.2, C120.2, C121.2, C38.2, C39.2, J5.3; no longer IC4.C1, IC4.GND
- net HEATER1: now also R50.1
- net HEATER2: now also R51.1
- net HEATER3: now also R52.1
- net SERVO: now also J5.1
- net SG_TST_E1: now also IC12-1.I3; no longer IC12-2.I1
- net SG_TST_E2: now also IC12-1.I2; no longer IC12-2.I2
- net SG_TST_E3: now also IC12-1.I1; no longer IC12-2.I3
- net SG_TST_X: now also IC12-2.I3; no longer IC12-1.I1
- net SG_TST_Y: now also IC12-2.I2; no longer IC12-1.I2
- net SG_TST_Z: now also IC12-2.I1; no longer IC12-1.I3
- net T_BED: now also C42.1, IC3.PB1/AD5, R37.1; no longer C44.1, IC3.PB0/AD4, R36.1
- net T_BED_IN: now also BED-2.S, R37.2, R41.1; no longer BED-1.S, R36.2, R43.1
- net T_EXT1_IN: now also EXT1-2.S; no longer EXT1-1.S
- net T_EXT2: now also C44.1, IC3.PB0/AD4, R36.1; no longer C42.1, IC3.PB1/AD5, R37.1
- net T_EXT2_IN: now also EXT2-2.S, R36.2, R43.1; no longer EXT2-1.S, R37.2, R41.1
- net T_EXT3_IN: now also EXT3-2.S; no longer EXT3-1.S
- net VSSA: now also BED-1.S, EXT1-1.S, EXT2-1.S, EXT3-1.S; no longer BED-2.S, EXT1-2.S, EXT2-2.S, EXT3-2.S
- net X_DIR: now also IC3.PA25/PGMD13; no longer IC3.PA7/XIN32/PGMNVALID
- net X_STOP: now also C120.1, D6.A2, R88.1; no longer X_STOP-1.S
- net Y_DIR: now also IC3.PA7/XIN32/PGMNVALID; no longer IC3.PA25/PGMD13
- net Y_STOP: now also C118.1, D4.A2, R86.1; no longer Y_STOP-1.S
- net Z_STOP: now also C38.1, D4.A1, R79.1; no longer IC4.OUT
- net Z_STOP_IN: now also R79.2, R95.1; no longer IC4.A1
Other:
- moved on the sheet: 3V3, 5V, BED-1, BED-2, C111, C112, C113, C114, C115, C116, C117, C15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
