File: projects/AMR3350/V7-32/AMR3350.sch (EAGLE design)
At the start: 241 parts, among them IC1 A4403, IC10 TMC5130, IC11 TMC5130, IC12 74LS32D, IC13 TMC5130, IC2 LDO-TS1117CW-3V3, IC3 ATSAM4S8C, IC5 74HC125, IC6 74S08D, IC7 TMC5130, IC8 TMC5130, J1 MOLEX-105162-001, J2 MSTBV4, Q1 NX138BKS, Q2 NX138BKS, Q3 AON7524, Q4 AON7524, X1 KK-254-4, X2 12MHz, X3 KK-254-2, X4 KK-254-4, X6 KK-254-4, X7 KK-254-4, X8 KK-254-4, X9 KK-254-4

Commit message: Forgot to save
Parts:
- renumbered X1 to MOT-E2, X3 to BEDOUT, X4 to MOT-Z1, X6 to MOT-X, X7 to MOT-Y, X8 to MOT-Z2, X9 to MOT-E1

Commit message: More progress
Connections:
- net A1_E3 renamed A1_E1
- net A1_E4 renamed A1_E2
- net A1_X1 renamed A1_X
- net A1_Y1 renamed A1_Y
- net A1_Z1 renamed A1_Z
- net A2_E3 renamed A2_E1
- net A2_E4 renamed A2_E2
- net A2_X1 renamed A2_X
- net A2_Y1 renamed A2_Y
- net A2_Z1 renamed A2_Z
- net A_Z2 renamed A_Z
- net B1_E3 renamed B1_E1
- net B1_E4 renamed B1_E2
- net B1_X1 renamed B1_X
- net B1_Y1 renamed B1_Y
- net B1_Z1 renamed B1_Z
- net B2_E3 renamed B2_E1
- net B2_E4 renamed B2_E2
- net B2_X1 renamed B2_X
- net B2_Y1 renamed B2_Y
- net B2_Z1 renamed B2_Z
- net B_Z2 renamed B_Z

Commit message: More more progress
Connections:
- net B1_Z: now also MOT-Z2-4.S; no longer MOT-Z1-3.S
- net B2_Z: now also MOT-Z1-3.S; no longer MOT-Z2-4.S
Changed lines of the file:
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@@
 <?xml version="1.0" encoding="utf-8"?>
 <!DOCTYPE eagle SYSTEM "eagle.dtd">
-<eagle version="9.4.1">
+<eagle version="9.5.0">
 <drawing>
 <settings>
@@
 <segment>
 <pinref part="C70" gate="G$1" pin="1"/>
-<wire x1="1668.78" y1="30.48" x2="1643.38" y2="30.48" width="0.1524" layer="91"/>
 <wire x1="1643.38" y1="30.48" x2="1638.3" y2="30.48" width="0.1524" layer="91"/>
 <wire x1="1643.38" y1="30.48" x2="1643.38" y2="27.94" width="0.1524" layer="91"/>
 <wire x1="1643.38" y1="27.94" x2="1645.92" y2="27.94" width="0.1524" layer="91"/>
-<junction x="1643.38" y="30.48"/>
 <pinref part="IC8" gate="G$1" pin="OB1"/>
-<pinref part="MOT-Z1" gate="-3" pin="S"/>
+<wire x1="1643.38" y1="30.48" x2="1661.16" y2="30.48" width="0.1524" layer="91"/>
+<junction x="1643.38" y="30.48"/>
+<pinref part="MOT-Z2" gate="-4" pin="S"/>
+<wire x1="1666.24" y1="22.86" x2="1678.94" y2="22.86" width="0.1524" layer="91"/>
+<wire x1="1661.16" y1="30.48" x2="1666.24" y2="22.86" width="0.1524" layer="91"/>
 </segment>
 </net>
@@
 <junction x="1643.38" y="25.4"/>
 <pinref part="IC8" gate="G$1" pin="OB2"/>
-<pinref part="MOT-Z2" gate="-4" pin="S"/>
-<wire x1="1663.7" y1="25.4" x2="1666.24" y2="22.86" width="0.1524" layer="91"/>
-<wire x1="1666.24" y1="22.86" x2="1678.94" y2="22.86" width="0.1524" layer="91"/>
+<wire x1="1663.7" y1="25.4" x2="1666.24" y2="30.48" width="0.1524" layer="91"/>
+<pinref part="MOT-Z1" gate="-3" pin="S"/>
+<wire x1="1666.24" y1="30.48" x2="1668.78" y2="30.48" width="0.1524" layer="91"/>
 </segment>
 </net>
