File: projects/AMR3350/V7-32/AMR3350.sch (EAGLE design)
At the start: 241 parts, among them IC1 A4403, IC10 TMC5130, IC11 TMC5130, IC12 74LS32D, IC13 TMC5130, IC2 LDO-TS1117CW-3V3, IC3 ATSAM4S8C, IC5 74HC125, IC6 74S08D, IC7 TMC5130, IC8 TMC5130, J1 MOLEX-105162-001, J2 MSTBV4, Q1 NX138BKS, Q2 NX138BKS, Q3 AON7524, Q4 AON7524, X2 12MHz

Commit message: Almost done?
Parts:
- added C72, C73, C74: (no value), resistor:C-EUC0603
- added D4, D5, D6: BAT54, diode:BAT54
- ERASE: value (none) -> J; device jumper:JP1Q -> con-other:J
Connections:
- net 24V_LED renamed 12V_LED
- removed net T_EXT_IN: EXT1-1.S, R37.2, R40.1
- new net T_EXT_IN2: EXT2-1.S, R38.2, R39.1
- net +12V: no longer R48.2, R49.2
- net +3V3: now also D4.C, D5.C, D6.C
- net E1_FUSED: now also R48.2
- net E2_FUSED: now also R49.2
- net GND: now also C72.2, C73.2, C74.2
- net T_EXT_IN1: now also EXT1-1.S, R37.2, R40.1; no longer EXT2-1.S, R38.2, R39.1
- net X_STOP: now also C73.1, D4.A
- net Y_STOP: now also C72.1, D5.A
- net Z_STOP: now also C74.1, D6.A
Other:
- moved on the sheet: EXT1_L, EXT2_L, J2-1, J2-2, J2-3, J2-4, R48, R49

Commit message: 20 parts left
Parts:
- added R51, R52, R53, R54, R55, R56: 10K, resistor:R-US_R0603
- C72, C73, C74: value (none) -> 2.2u
Connections:
- new net X_STOP_IN: R51.2, R56.1, X_STOP-1.S
- new net Y_STOP_IN: R52.2, R55.1, Y_STOP-1.S
- new net Z_STOP_IN: R53.2, R54.1, Z_STOP-1.S
- net +3V3: now also R54.2, R55.2, R56.2
- net EXT1: no longer IC3.PA20/PGMD8/AD3
- net FAN_PART: no longer IC3.PC13/AD10
- net X_DIR: now also IC3.PC13/AD10; no longer IC3.PA16/PGMD4
- net X_EN: now also IC3.PA20/PGMD8/AD3; no longer IC3.PA15/PGMD3
- net X_STEP: now also IC3.PC12/AD12; no longer IC3.PC7
- net X_STOP: now also IC3.PA15/PGMD3, R51.1; no longer IC3.PC16, X_STOP-1.S
- net Y_STOP: now also IC3.PC7, R52.1; no longer IC3.PA0/PGMEN0, Y_STOP-1.S
- net Z_STOP: now also IC3.PA16/PGMD4, R53.1; no longer IC3.PC17, Z_STOP-1.S
Other:
- moved on the sheet: C72, C73, C74, D4, D5, D6, X_STOP-1, X_STOP-2, X_STOP-3, Z_STOP-1, Z_STOP-2, Z_STOP-3

Commit message: 66 airwires left
Parts:
- removed IC6: 74S08D, 74xx-us:74S08D
- added IC4: 74ABT125BQ, 74xx-us:74ABT125BQ
- added R57: 4K7, resistor:R-US_R0603
- IC5: value 74HC125 -> 74AHC08; device misc:74HC125 -> misc:74AHC08
Connections:
- net FAN_MOBO renamed FAN_3
- removed net FAN_E1: IC3.PC3, R42.1
- removed net FAN_E2: IC3.PC0, R43.1
- removed net FAN_PART: R45.1
- new net FAN_1: IC3.TDO/TRACESWO/PB5, R42.1
- new net FAN_2: IC3.PC2, R43.1
- new net FAN_4: IC3.PA0/PGMEN0, R45.1
- net +3V3: now also IC4P.VCC; no longer IC5P.VCC
- net +5V: now also IC5P.VCC; no longer IC6P.VCC
- net ENN: now also IC3.PC0; no longer IC3.PC14
- net ESP_DATA_RDY: now also IC3.PC16; no longer IC3.PC26
- net ESP_EN: now also IC3.PC14; no longer IC3.PC6
- net ESP_RESET: now also IC3.PC6; no longer IC3.PC2
- net EXT1: now also IC3.PC3
- net GND: now also IC4A.I, IC4A.OE, IC4C.OE, IC4D.OE, IC4P.GND, IC5A.I0, IC5A.I1, R57.1; no longer IC5A.OE, IC5B.OE, IC5D.I, IC5D.OE, IC6C.I0, IC6C.I1, IC6P.GND
- net LCD_BEEP: now also IC3.PC17, R57.2; no longer IC3.PC23
- net LCD_CS: now also IC5B.I1, IC5C.I0, IC5C.I1, IC5D.I0; no longer IC6A.I1, IC6B.I0, IC6B.I1, IC6D.I1
- net LCD_CS_BUF: now also IC5C.O; no longer IC6B.O
- net LCD_MISO: now also IC4B.O; no longer IC5C.O
- net LCD_MISO_BUF: now also IC4B.I; no longer IC5C.I
- net LCD_MOSI: now also IC4C.I, IC5B.I0; no longer IC5A.I, IC6A.I0
- net LCD_MOSI_BUF: now also IC5B.O; no longer IC6A.O
- net LCD_SCK: now also IC4D.I, IC5D.I1; no longer IC5B.I, IC6D.I0
- net LCD_SCK_BUF: now also IC5D.O; no longer IC6D.O
- net LCD_SD_CS: now also IC4B.OE; no longer IC5C.OE
- net SAM_TFR_RDY: now also IC3.PA1/PGMEN1; no longer IC3.PA7/XIN32/PGMNVALID
- net SD_MOSI_BUF: now also IC4C.O; no longer IC5A.O
- net SD_SCK_BUF: now also IC4D.O; no longer IC5B.O
- net SG_TST: now also IC3.PA7/XIN32/PGMNVALID; no longer IC3.PA1/PGMEN1
Other:
- moved on the sheet: IC5P

Commit message: Done!
Parts:
- removed C125, C128, C129, C130, C132: 100n, resistor:C-EUC0603
- removed C126: 4u7, resistor:C-EUC0603
- removed C127: 470n, resistor:C-EUC0603
- removed C131: 22n, resistor:C-EUC0603
- removed C133: 100u, resistor:CPOL-USD
- removed C134, C135, C136, C137: 470p, resistor:C-EUC0402
- removed IC12: 74LS32D, 74xx-us:74LS32D
- removed R82, R83: 0R11, resistor:R-US_R1206
- removed R84: 20K, resistor:R-TRIMM3103
- removed R85: 20K, resistor:R-US_R0603
- added C112, C113, C84: 470p, resistor:C-EUC0402
- added C114: 100n, rcl:C-EUC0603
- added C75, C78, C79, C82, C83: 100n, resistor:C-EUC0603
- added C76: 470n, resistor:C-EUC0603
- added C77: 4u7, resistor:C-EUC0603
- added C80: 22n, resistor:C-EUC0603
- added C81: 100u, resistor:CPOL-USD
- added IC9: TMC5130, TMC5130_3D_Printer_BOARD_V_2:TMC5130
- added R66, R67: 0R11, resistor:R-US_R1206
- added R68: 20K, resistor:R-TRIMM3103
- added R69: 20K, resistor:R-US_R0603
- C100, C61, C87: value 470n -> 470p; device resistor:C-EUC0603 -> resistor:C-EUC0402
- C102, C50, C63, C89: value 100n -> 470n
- C103, C51, C64, C90: value 100n -> 4u7
- C104, C52, C65, C91: value 22n -> 100n
- C106, C54, C67, C93: value 100u -> 22n; device resistor:CPOL-USD -> resistor:C-EUC0603
- C107, C55, C68, C94: value 470p -> 100u; device resistor:C-EUC0402 -> resistor:CPOL-USD
- C108, C109, C56, C57, C69, C70, C95, C96: value 470p -> 100n; device resistor:C-EUC0402 -> resistor:C-EUC0603
- C111: value 100n -> 470p; device rcl:C-EUC0603 -> resistor:C-EUC0402
- C45, C46: value 100n -> 2.2u
- C47: value 4u7 -> 2.2u
- C48: value 470n -> 100n
- C59, C85, C98: value 100n -> 470p; device resistor:C-EUC0603 -> resistor:C-EUC0402
- C60, C86, C99: value 4u7 -> 470p; device resistor:C-EUC0603 -> resistor:C-EUC0402
- C72, C73, C74: value 2.2u -> 470p; device resistor:C-EUC0603 -> resistor:C-EUC0402
- IC11: value TMC5130 -> 74LS32D; device TMC5130_3D_Printer_BOARD_V_2:TMC5130 -> 74xx-us:74LS32D
- R39, R40, R41: value 4K7 0.1% -> 10K
- R42, R43, R44: value 1K -> 10K
- R45: value 1K -> 4K7 0.1%
- R46, R47: value 180R -> 4K7 0.1%
- R48, R49: value 4K7 -> 1K
- R50: value 180R -> 1K
- R51: value 10K -> 1K
- R52, R53, R56: value 10K -> 180R
- R54, R55: value 10K -> 4K7
- renumbered 3V3 to 3V1, IC13 to IC6, X2 to X1
Connections:
- net +12V: now also C104.2, C107.+, C108.1, C109.1, C52.2, C55.+, C56.1, C57.1, C65.2, C68.+, C69.1, C70.1, C78.2, C79.1, C81.+, C82.1, C83.1, C91.2, C94.+, C95.1, C96.1, IC9.VS, IC9.VSA; no longer C101.2, C102.1, C103.1, C106.+, C128.2, C129.1, C130.1, C132.1, C133.+, C49.2, C50.1, C51.1, C54.+, C62.2, C63.1, C64.1, C67.+, C88.2, C89.1, C90.1, C93.+, IC11.VS, IC11.VSA
- net +3V3: now also C101.1, C114.1, C47.1, C49.1, C62.1, C75.1, C88.1, IC11P.VCC, IC9.VCC_IO, R39.2, R40.2, R41.2; no longer C111.1, C125.1, C44.1, C46.1, C59.1, C85.1, C98.1, IC11.VCC_IO, IC12P.VCC, R54.2, R55.2, R56.2
- net +5V: now also C102.1, C50.1, C63.1, C76.1, C89.1, IC9.VCC, R69.2; no longer C100.1, C127.1, C45.1, C61.1, C87.1, IC11.VCC, R85.2
- net 5V_E1: now also C51.1; no longer C126.1
- net 5V_E2: now also C64.1; no longer C47.1
- net 5V_X: now also C77.1, IC8.5VOUT; no longer C86.1, IC10.5VOUT
- net 5V_Y: now also C90.1, IC9.5VOUT; no longer C99.1, IC11.5VOUT
- net 5V_Z: now also C103.1, IC10.5VOUT; no longer C60.1, IC8.5VOUT
- net A1_E1: now also C58.1; no longer C134.1
- net A1_E2: now also C71.1; no longer C55.1
- net A1_X: now also C84.1, IC8.OA1; no longer C94.1, IC10.OA1
- net A1_Y: now also C97.1, IC9.OA1; no longer C107.1, IC11.OA1
- net A1_Z: now also C110.1, IC10.OA1; no longer C68.1, IC8.OA1
- net A2_E1: now also C59.1; no longer C135.1
- net A2_E2: now also C72.1; no longer C56.1
- net A2_X: now also C85.1, IC8.OA2; no longer C95.1, IC10.OA2
- net A2_Y: now also C98.1, IC9.OA2; no longer C108.1, IC11.OA2
- net A2_Z: now also C111.1, IC10.OA2; no longer C69.1, IC8.OA2
- net ADVREF: now also R45.2, R46.2, R47.2; no longer R39.2, R40.2, R41.2
- net B1_E1: now also C60.1; no longer C136.1
- net B1_E2: now also C73.1; no longer C57.1
- net B1_X: now also C86.1, IC8.OB1; no longer C96.1, IC10.OB1
- net B1_Y: now also C99.1, IC9.OB1; no longer C109.1, IC11.OB1
- net B1_Z: now also C112.1, IC10.OB1; no longer C70.1, IC8.OB1
- net B2_E1: now also C61.1; no longer C137.1
- net B2_E2: now also C74.1; no longer C58.1
- net B2_X: now also C87.1, IC8.OB2; no longer C97.1, IC10.OB2
- net B2_Y: now also C100.1, IC9.OB2; no longer C110.1, IC11.OB2
- net B2_Z: now also C113.1, IC10.OB2; no longer C71.1, IC8.OB2
- net BED: now also R56.1; no longer R50.1
- net BED_L: now also R55.1; no longer R49.1
- net BED_OUT: now also R56.2; no longer R50.2
- net BRA_E1: now also R58.1; no longer R82.1
- net BRA_E2: now also R62.1; no longer R58.1
- net BRA_X: now also IC8.BRA, R66.1; no longer IC10.BRA, R70.1
- net BRA_Y: now also IC9.BRA, R70.1; no longer IC11.BRA, R74.1
- net BRA_Z: now also IC10.BRA, R74.1; no longer IC8.BRA, R62.1
- net BRB_E1: now also R59.1; no longer R83.1
- net BRB_E2: now also R63.1; no longer R59.1
- net BRB_X: now also IC8.BRB, R67.1; no longer IC10.BRB, R71.1
- net BRB_Y: now also IC9.BRB, R71.1; no longer IC11.BRB, R75.1
- net BRB_Z: now also IC10.BRB, R75.1; no longer IC8.BRB, R63.1
- net CPI_E1: now also C54.1; no longer C131.1
- net CPI_E2: now also C67.1; no longer C52.1
- net CPI_X: now also C80.1, IC8.CPI; no longer C91.1, IC10.CPI
- net CPI_Y: now also C93.1, IC9.CPI; no longer C104.1, IC11.CPI
- net CPI_Z: now also C106.1, IC10.CPI; no longer C65.1, IC8.CPI
- net CPO_E1: now also C54.2; no longer C131.2
- net CPO_E2: now also C67.2; no longer C52.2
- net CPO_X: now also C80.2, IC8.CPO; no longer C91.2, IC10.CPO
- net CPO_Y: now also C93.2, IC9.CPO; no longer C104.2, IC11.CPO
- net CPO_Z: now also C106.2, IC10.CPO; no longer C65.2, IC8.CPO
- net E1_FUSED: now also R54.2; no longer R48.2
- net E2_FUSED: now also R55.2; no longer R49.2
- net ENN: now also IC9.DRV_ENN_CFG6; no longer IC11.DRV_ENN_CFG6
- net EXT1: now also R52.1; no longer R46.1
- net EXT1_G: now also R52.2; no longer R46.2
- net EXT2: now also R53.1; no longer R47.1
- net EXT2_G: now also R53.2; no longer R47.2
- net EXT_L: now also R54.1; no longer R48.1
- net FAN1_G: now also R48.2; no longer R42.2
- net FAN2_G: now also R49.2; no longer R43.2
- net FAN3_G: now also R50.2; no longer R44.2
- net FAN4_G: now also R51.2; no longer R45.2
- net FAN_1: now also R48.1; no longer R42.1
- net FAN_2: now also R49.1; no longer R43.1
- net FAN_3: now also R50.1; no longer R44.1
- net FAN_4: now also R51.1; no longer R45.1
- net GND: now also C101.2, C104.1, C107.-, C112.2, C113.2, C114.2, C49.2, C52.1, C55.-, C62.2, C65.1, C68.-, C75.2, C76.2, C77.2, C78.1, C81.-, C82.2, C83.2, C84.2, C88.2, C91.1, C94.-, IC11P.GND, IC9.CLK, IC9.ENCB_DCEN_CFG4, IC9.GND, IC9.GNDA, IC9.GNDP, IC9.GND_PAD, IC9.TST_MODE, R66.2, R67.2, R68.A; no longer C101.1, C106.-, C107.2, C125.2, C126.2, C127.2, C128.1, C129.2, C130.2, C133.-, C134.2, C135.2, C136.2, C137.2, C49.1, C54.-, C55.2, C62.1, C67.-, C68.2, C88.1, C93.-, C94.2, IC11.CLK, IC11.ENCB_DCEN_CFG4, IC11.GND, IC11.GNDA, IC11.GNDP, IC11.GND_PAD, IC11.TST_MODE, IC12P.GND, R82.2, R83.2, R84.A
- net IREF_E1: now also R60.S; no longer R84.S
- net IREF_E2: now also R64.S; no longer R60.S
- net IREF_X: now also IC8.AIN_IREF, R68.S; no longer IC10.AIN_IREF, R72.S
- net IREF_Y: now also IC9.AIN_IREF, R72.S; no longer IC11.AIN_IREF, R76.S
- net IREF_Z: now also IC10.AIN_IREF, R76.S; no longer IC8.AIN_IREF, R64.S
- net MOT_MISO: now also IC9.SDO_NAO_CFG0; no longer IC11.SDO_NAO_CFG0
- net MOT_MOSI: now also IC9.SDI_NAI_CFG1; no longer IC11.SDI_NAI_CFG1
- net MOT_SCK: now also IC9.SCK_CFG2; no longer IC11.SCK_CFG2
- net REFIN_E1: now also R60.E, R61.1; no longer R84.E, R85.1
- net REFIN_E2: now also R64.E, R65.1; no longer R60.E, R61.1
- net REFIN_X: now also R68.E, R69.1; no longer R72.E, R73.1
- net REFIN_Y: now also R72.E, R73.1; no longer R76.E, R77.1
- net REFIN_Z: now also R76.E, R77.1; no longer R64.E, R65.1
- net SG_TST: now also IC11B.O; no longer IC12B.O
- net SG_TST_E1: now also IC11D.I0; no longer IC12D.I0
- net SG_TST_E1X: now also IC11C.I1, IC11D.O; no longer IC12C.I1, IC12D.O
- net SG_TST_E2: now also IC11C.I0; no longer IC12C.I0
- net SG_TST_EX: now also IC11B.I1, IC11C.O; no longer IC12B.I1, IC12C.O
- net SG_TST_X: now also IC11D.I1, IC8.SWP_DIAG1; no longer IC10.SWP_DIAG1, IC12D.I1
- net SG_TST_Y: now also IC11A.I0, IC9.SWP_DIAG1; no longer IC11.SWP_DIAG1, IC12A.I0
- net SG_TST_YZ: now also IC11A.O, IC11B.I0; no longer IC12A.O, IC12B.I0
- net SG_TST_Z: now also IC10.SWP_DIAG1, IC11A.I1; no longer IC12A.I1, IC8.SWP_DIAG1
- net T_BED: now also C46.1, R42.1; no longer C43.1, R36.1
- net T_BED_IN: now also R42.2, R47.1; no longer R36.2, R41.1
- net T_EXT1: now also C45.1, R43.1; no longer C42.1, R37.1
- net T_EXT2: now also C44.1, R44.1; no longer C41.1, R38.1
- net T_EXT_IN1: now also R43.2, R46.1; no longer R37.2, R40.1
- net T_EXT_IN2: now also R44.2, R45.1; no longer R38.2, R39.1
- net VCP_E1: now also C53.2; no longer C132.2
- net VCP_E2: now also C66.2; no longer C53.2
- net VCP_X: now also C79.2, IC8.VCP; no longer C92.2, IC10.VCP
- net VCP_Y: now also C92.2, IC9.VCP; no longer C105.2, IC11.VCP
- net VCP_Z: now also C105.2, IC10.VCP; no longer C66.2, IC8.VCP
- net X_DIR: now also IC8.REFR_DIR; no longer IC10.REFR_DIR
- net X_EN: now also IC8.CSN_CFG3; no longer IC10.CSN_CFG3
- net X_STEP: now also IC8.REFL_STEP; no longer IC10.REFL_STEP
- net X_STOP: now also C41.1, R36.1; no longer C73.1, R51.1
- net X_STOP_IN: now also R36.2, R39.1; no longer R51.2, R56.1
- net Y_DIR: now also IC9.REFR_DIR; no longer IC11.REFR_DIR
- net Y_EN: now also IC9.CSN_CFG3; no longer IC11.CSN_CFG3
- net Y_STEP: now also IC9.REFL_STEP; no longer IC11.REFL_STEP
- net Y_STOP: now also C42.1, R37.1; no longer C72.1, R52.1
- net Y_STOP_IN: now also R37.2, R40.1; no longer R52.2, R55.1
- net Z_DIR: now also IC10.REFR_DIR; no longer IC8.REFR_DIR
- net Z_EN: now also IC10.CSN_CFG3; no longer IC8.CSN_CFG3
- net Z_STEP: now also IC10.REFL_STEP; no longer IC8.REFL_STEP
- net Z_STOP: now also C43.1, R38.1; no longer C74.1, R53.1
- net Z_STOP_IN: now also R38.2, R41.1; no longer R53.2, R54.1
Other:
- moved on the sheet: C100, C101, C102, C103, C104, C105, C108, C109, C110, C111, C41, C42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

Commit message: Final** version of AMRV7/EE4SR1.1.1, new APSR
Parts:
- renumbered 3V1 to +3V3, 5V to +5V, EXP_1 to EXP1, EXP_2 to EXP2
