File: projects/AMR3350/V7-32/AMR3350.brd (EAGLE design)
At the start: 160 x 87 mm, 241 parts, among them IC1 A4403, IC10 TMC5130, IC11 TMC5130, IC12 74LS32D, IC13 TMC5130, IC2 LDO-TS1117CW-3V3, IC3 ATSAM4S8C, IC5 74HC125, IC6 74S08D, IC7 TMC5130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

Commit message: Forgot to save
Parts:
- removed X4, X8: KK-254-4, con-other:MOLEX-KK-254-4
- added MOT-Z1, MOT-Z2: KK-254-4, con-other:MOLEX-KK-254-4
- moved EXP_1 262.4 mm to (155.0, 29.5), turned to 90 degrees
- moved IC8 252.1 mm to (130.0, 61.5), turned to 45 degrees
- moved IC6 235.8 mm to (146.0, 47.5), turned to 90 degrees
- moved C22 192.5 mm to (92.5, 90.0)
- moved EXP_2 179.7 mm to (155.0, 51.0), turned to 90 degrees
- moved IC5 169.4 mm to (146.0, 33.5), turned to 90 degrees
- moved ESP8266 162.9 mm to (6.00, 77.5), turned to 90 degrees
- moved C23 161.4 mm to (92.5, 96.5)
- moved C24 161.4 mm to (86.0, 96.5)
- moved C27 161.4 mm to (79.5, 96.5)
- moved C28 161.4 mm to (73.5, 96.5)
- moved C29 161.4 mm to (67.0, 96.5)
- moved C30 161.4 mm to (60.5, 96.5)
- moved C31 161.4 mm to (54.5, 96.5)
- moved C33 161.4 mm to (48.0, 96.5)
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- renumbered X1 to MOT-E2, X3 to BEDOUT, X6 to MOT-X, X7 to MOT-Y, X9 to MOT-E1
Connections:
- net A1_Z1: now also MOT-Z2.1; no longer X8.1
- net A2_Z1: now also MOT-Z1.2; no longer X4.2
- net A_Z2: now also MOT-Z1.1, MOT-Z2.2; no longer X4.1, X8.2
- net B1_Z1: now also MOT-Z1.3; no longer X4.3
- net B2_Z1: now also MOT-Z2.4; no longer X8.4
- net B_Z2: now also MOT-Z1.4, MOT-Z2.3; no longer X4.4, X8.3
Routing:
- net GND: track 0.00 -> 81.7 mm
- net +12V: track 0.00 -> 64.6 mm
- net E2_FUSED: track 0.00 -> 10.5 mm
- net E1_FUSED: track 0.00 -> 10.5 mm
- net FAN3_D: track 0.00 -> 5.57 mm
- net FAN1_D: track 0.00 -> 5.57 mm
- net Z_STEP: track 0.00 -> 3.12 mm
- net Z_EN: track 0.00 -> 3.12 mm
- net Z_DIR: track 0.00 -> 3.12 mm
- net Y_STEP: track 0.00 -> 3.12 mm
- net Y_EN: track 0.00 -> 3.12 mm
- net Y_DIR: track 0.00 -> 3.12 mm
- net X_STEP: track 0.00 -> 3.12 mm
- net X_EN: track 0.00 -> 3.12 mm
- net X_DIR: track 0.00 -> 3.12 mm
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- added copper zone on layer 1, net EXT1_D
- added copper zone on layer 16, net EXT1_D
- added copper zone on layer 1, net EXT2_D
- added copper zone on layer 16, net EXT2_D
- added copper zone on layer 1, net GND

Commit message: Progress
Parts:
- moved R63 226.1 mm to (111.7, 58.5), turned to 270 degrees
- moved R64 213.8 mm to (107.4, 69.1), turned to 135 degrees
- moved C67 208.6 mm to (92.5, 59.5), turned to 90 degrees
- moved R62 205.4 mm to (97.3, 58.5), turned to 270 degrees
- moved C65 191.3 mm to (100.0, 65.8), turned to 45 degrees
- moved C60 189.4 mm to (103.7, 67.8), turned to 90 degrees
- moved C66 185.8 mm to (97.6, 63.5), turned to 90 degrees
- moved C63 184.6 mm to (109.8, 65.0), turned to 135 degrees
- moved C64 177.9 mm to (96.6, 66.1)
- moved C71 177.4 mm to (109.1, 71.2), turned to 315 degrees
- moved R2 169.0 mm to (19.5, -8.50), turned to 270 degrees
- moved C59 168.6 mm to (109.0, 55.4)
- moved C70 167.9 mm to (105.5, 72.0), turned to 180 degrees
- moved C62 165.2 mm to (95.6, 63.5), turned to 90 degrees
- moved C61 163.1 mm to (100.9, 68.6), turned to 180 degrees
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Routing:
- net GND: track 81.7 -> 397.3 mm, vias 0 -> 42
- net GND3: track 0.00 -> 92.0 mm, vias 0 -> 34
- net GND2: track 0.00 -> 92.0 mm, vias 0 -> 34
- net GND1: track 0.00 -> 92.0 mm, vias 0 -> 34
- net +12V: track 64.6 -> 102.0 mm, vias 0 -> 4
- net A1_Z4: track 0.00 -> 34.9 mm, vias 0 -> 3
- net A1_Z3: track 0.00 -> 34.9 mm, vias 0 -> 3
- net A1_Z2: track 0.00 -> 34.9 mm, vias 0 -> 3
- net A1_Z1: track 0.00 -> 34.9 mm, vias 0 -> 3
- net LX: track 0.00 -> 28.1 mm
- net B2_Z4: track 0.00 -> 27.8 mm, vias 0 -> 3
- net B2_Z3: track 0.00 -> 27.8 mm, vias 0 -> 3
- net B2_Z2: track 0.00 -> 27.8 mm, vias 0 -> 3
- net B2_Z1: track 0.00 -> 27.8 mm, vias 0 -> 3
- net B1_Z2: track 0.00 -> 27.4 mm, vias 0 -> 2
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- added copper zone on layer 1, net +3V3
- added copper zone on layer 16, net +3V3
- added copper zone on layer 1, net LX
- added copper zone on layer 1, net VOUT
Other:
- board size 160 x 87 mm -> 115 x 87 mm

Commit message: More progress
Parts:
- moved C46 239.0 mm to (109.0, 61.9)
- moved R61 232.7 mm to (103.9, 76.9), turned to 180 degrees
- moved C136 215.6 mm to (89.1, 77.7), turned to 315 degrees
- moved R84 214.8 mm to (87.4, 75.6), turned to 135 degrees
- moved R59 213.0 mm to (111.7, 65.0), turned to 270 degrees
- moved IC7 212.8 mm to (104.5, 67.5), turned to 90 degrees
- moved R60 204.8 mm to (107.4, 75.6), turned to 135 degrees
- moved C135 202.2 mm to (81.7, 77.7), turned to 270 degrees
- moved C54 202.0 mm to (95.5, 78.0), turned to 270 degrees
- moved MOT-E2 200.2 mm to (104.5, 82.5)
- moved C134 193.6 mm to (79.5, 77.7), turned to 270 degrees
- moved R58 192.2 mm to (97.3, 65.0), turned to 270 degrees
- moved C92 182.2 mm to (57.6, 70.0), turned to 90 degrees
- moved C98 181.8 mm to (49.0, 61.9)
- moved R72 180.9 mm to (67.4, 75.6), turned to 135 degrees
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Connections:
- net A1_E3 renamed A1_E1
- net A1_E4 renamed A1_E2
- net A1_X1 renamed A1_X
- net A1_Y1 renamed A1_Y
- net A1_Z1 renamed A1_Z
- net A2_E3 renamed A2_E1
- net A2_E4 renamed A2_E2
- net A2_X1 renamed A2_X
- net A2_Y1 renamed A2_Y
- net A2_Z1 renamed A2_Z
- net A_Z2 renamed A_Z
- net B1_E3 renamed B1_E1
- net B1_E4 renamed B1_E2
- net B1_X1 renamed B1_X
- net B1_Y1 renamed B1_Y
- net B1_Z1 renamed B1_Z
- net B2_E3 renamed B2_E1
- net B2_E4 renamed B2_E2
- net B2_X1 renamed B2_X
- net B2_Y1 renamed B2_Y
- net B2_Z1 renamed B2_Z
- net B_Z2 renamed B_Z
Routing:
- net GND: track 397.3 -> 721.3 mm, vias 42 -> 144
- net +12V: track 102.0 -> 311.3 mm, vias 4 -> 8
- net GND3: track 92.0 -> 0.00 mm, vias 34 -> 0
- net GND2: track 92.0 -> 0.00 mm, vias 34 -> 0
- net GND1: track 92.0 -> 0.00 mm, vias 34 -> 0
- net ENN: track 19.4 -> 77.5 mm
- net A1_Z4: track 34.9 -> 0.00 mm, vias 3 -> 0
- net A1_Z3: track 34.9 -> 0.00 mm, vias 3 -> 0
- net A1_Z2: track 34.9 -> 0.00 mm, vias 3 -> 0
- net A1_Z: track 34.9 -> 0.00 mm, vias 3 -> 0
- net A1_Y: track 0.00 -> 29.0 mm, vias 0 -> 2
- net A1_X: track 0.00 -> 29.0 mm, vias 0 -> 2
- net A1_E2: track 0.00 -> 29.0 mm, vias 0 -> 2
- net A1_E1: track 0.00 -> 29.0 mm, vias 0 -> 2
- net B1_Y: track 0.00 -> 27.9 mm, vias 0 -> 2
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
Commit message: More more progress
Parts:
- moved C71 28.0 mm to (9.10, 89.2)
- moved R63 21.3 mm to (31.2, 71.5)
- moved C59 21.3 mm to (28.5, 68.4)
- moved C60 21.3 mm to (23.2, 80.8)
- moved C61 21.3 mm to (20.4, 81.6)
- moved C63 21.3 mm to (29.3, 78.0)
- moved C65 21.3 mm to (19.5, 78.8)
- moved C66 21.3 mm to (17.1, 76.5)
- moved R62 21.3 mm to (16.8, 71.5)
- moved R65 21.3 mm to (23.4, 83.4)
- moved R64 21.0 mm to (27.2, 82.3), turned to 90 degrees
- moved C64 19.9 mm to (17.1, 80.4)
- moved C62 15.1 mm to (17.1, 82.5), turned to 180 degrees
- moved C14 2.24 mm to (18.6, 65.3), turned to 0 degrees
Connections:
- net B1_Z: now also MOT-Z2.4; no longer MOT-Z1.3
- net B2_Z: now also MOT-Z1.3; no longer MOT-Z2.4
Routing:
- net +5V: track 51.3 -> 215.8 mm, vias 0 -> 4
- net GND: track 721.3 -> 801.2 mm, vias 144 -> 175
- net B1_Z: track 0.00 -> 43.2 mm, vias 0 -> 2
- net B2_Z: track 0.00 -> 30.2 mm, vias 0 -> 2
- net +12V: track 311.3 -> 334.2 mm, vias 8 -> 7
- net A1_Z: track 0.00 -> 19.0 mm, vias 0 -> 2
- net SG_TST_Z: track 0.00 -> 17.1 mm
- net ENN: track 77.5 -> 93.5 mm
- net E1_FUSED: track 0.06 -> 11.5 mm
- net E2_FUSED: track 0.17 -> 11.5 mm
- net A2_Z: track 0.00 -> 11.4 mm, vias 0 -> 2
- net IREF_Z: track 0.00 -> 4.78 mm
- net REFIN_Z: track 0.00 -> 4.22 mm
- net VCP_Z: track 0.00 -> 3.16 mm
- net BRB_Z: track 0.00 -> 3.14 mm
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
Commit message: More progress
Parts:
- moved C68 39.0 mm to (8.90, 68.6), turned to 0 degrees
- moved C69 38.1 mm to (14.2, 68.6), turned to 0 degrees
- moved C70 24.5 mm to (30.0, 81.5), turned to 90 degrees
- moved C71 15.1 mm to (15.5, 75.5), turned to 270 degrees
- moved D3 10.8 mm to (75.0, 11.5)
- moved IC3 5.63 mm to (76.4, 32.9), turned to 225 degrees
- moved J1 5.00 mm to (109.0, 25.5)
- moved C66 1.10 mm to (17.0, 77.6), turned to 315 degrees
Routing:
- net GND: track 801.2 -> 981.8 mm, vias 175 -> 180
- net +3V3: track 21.4 -> 111.6 mm
- net Z_EN: track 3.12 -> 60.0 mm
- net Z_DIR: track 3.13 -> 59.2 mm
- net Z_STEP: track 3.13 -> 57.8 mm
- net Y_EN: track 3.12 -> 39.1 mm
- net Y_STEP: track 3.13 -> 37.1 mm
- net Y_DIR: track 3.13 -> 36.8 mm
- net X_EN: track 3.13 -> 26.5 mm
- net X_STEP: track 3.13 -> 25.3 mm
- net X_DIR: track 3.13 -> 24.9 mm
- net USB_P: track 0.00 -> 7.83 mm
- net USB_N: track 0.00 -> 7.81 mm
- net VBUS: track 0.00 -> 5.60 mm, vias 0 -> 1
- net A1_Z: track 19.0 -> 23.6 mm
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
Commit message: More progress
Parts:
- moved IC12 160.0 mm to (59.0, 54.5), turned to 270 degrees
- moved X2 146.5 mm to (78.7, 23.5), turned to 315 degrees
- moved C17 88.1 mm to (64.1, 40.9), turned to 270 degrees
- moved C21 84.7 mm to (51.0, 45.5)
- moved C32 83.8 mm to (75.6, 39.9), turned to 90 degrees
- moved C18 83.8 mm to (55.5, 32.5), turned to 270 degrees
- moved C23 78.1 mm to (79.0, 35.7), turned to 45 degrees
- moved C25 72.3 mm to (77.0, 34.0), turned to 315 degrees
- moved C34 71.3 mm to (76.1, 36.8)
- moved C33 68.9 mm to (77.7, 39.4), turned to 90 degrees
- moved C19 65.2 mm to (62.0, 19.2), turned to 90 degrees
- moved C36 62.1 mm to (69.0, 26.5)
- moved C37 62.1 mm to (64.0, 26.5)
- moved C20 51.9 mm to (78.1, 19.8), turned to 135 degrees
- moved IC3 10.1 mm to (67.0, 29.0)
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Connections:
- removed net SG_TST_E1Z: IC12.10, IC12.6
- removed net SG_TST_XY: IC12.12, IC12.3
- removed net SG_TST_ZE: IC12.13, IC12.8
- new net SG_TST_E1X: IC12.10, IC12.11
- new net SG_TST_EX: IC12.5, IC12.8
- new net SG_TST_YZ: IC12.3, IC12.4
- net SG_TST: now also IC12.6; no longer IC12.11
- net SG_TST_E1: now also IC12.12; no longer IC12.5
- net SG_TST_X: now also IC12.13; no longer IC12.1
- net SG_TST_Y: now also IC12.1; no longer IC12.2
- net SG_TST_Z: now also IC12.2; no longer IC12.4
Routing:
- net GND: track 981.8 -> 1316.7 mm, vias 180 -> 236
- net MOT_MISO: track 0.00 -> 143.8 mm, vias 0 -> 6
- net MOT_SCK: track 0.00 -> 140.8 mm, vias 0 -> 5
- net MOT_MOSI: track 0.00 -> 140.0 mm, vias 0 -> 5
- net ENN: track 93.5 -> 210.0 mm, vias 0 -> 4
- net SG_TST_E2: track 16.9 -> 80.6 mm, vias 0 -> 2
- net +3V3: track 111.6 -> 166.1 mm, vias 6 -> 11
- net SG_TST_E1: track 16.9 -> 61.6 mm, vias 0 -> 2
- net Z_EN: track 60.0 -> 17.3 mm
- net SG_TST_Z: track 17.1 -> 58.0 mm, vias 0 -> 2
- net Z_DIR: track 59.2 -> 18.7 mm
- net Z_STEP: track 57.8 -> 18.7 mm
- net Y_EN: track 39.1 -> 11.3 mm
- net Y_DIR: track 36.8 -> 9.30 mm
- net Y_STEP: track 37.1 -> 9.74 mm
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
Commit message: Almost done?
Parts:
- added C72, C73, C74: (no value), resistor:C0603
- added D4, D5, D6: BAT54, diode:SOT23
- ERASE: value (none) -> J; device jumper:JP1 -> con-other:1X02
- moved C44 287.3 mm to (151.0, 31.5)
- moved C45 285.0 mm to (155.0, 31.5)
- moved C41 250.5 mm to (135.5, 59.0)
- moved C42 250.5 mm to (130.5, 59.0)
- moved C43 250.5 mm to (125.5, 59.0)
- moved R41 237.2 mm to (125.5, 54.0)
- moved R38 234.3 mm to (135.5, 56.5)
- moved R40 232.3 mm to (130.5, 54.0)
- moved BED 228.7 mm to (111.0, 39.5), turned to 270 degrees
- moved R39 227.4 mm to (135.5, 54.0)
- moved R37 224.8 mm to (130.5, 56.5)
- moved R14 220.6 mm to (80.5, 37.9), turned to 315 degrees
- moved C40 217.3 mm to (92.8, 23.7), turned to 180 degrees
- moved R13 215.9 mm to (66.9, 11.5), turned to 270 degrees
- moved R36 215.4 mm to (125.5, 56.5)
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Connections:
- net 24V_LED renamed 12V_LED
- removed net T_EXT_IN: EXT1.1, R37.2, R40.1
- new net T_EXT_IN2: EXT2.1, R38.2, R39.1
- net +12V: no longer R48.2, R49.2
- net +3V3: now also D4.3, D5.3, D6.3
- net E1_FUSED: now also R48.2
- net E2_FUSED: now also R49.2
- net GND: now also C72.2, C73.2, C74.2
- net T_EXT_IN1: now also EXT1.1, R37.2, R40.1; no longer EXT2.1, R38.2, R39.1
- net X_STOP: now also C73.1, D4.1
- net Y_STOP: now also C72.1, D5.1
- net Z_STOP: now also C74.1, D6.1
Routing:
- net GND: track 1316.7 -> 1523.3 mm, vias 236 -> 259
- net +3V3: track 166.1 -> 325.3 mm, vias 11 -> 35
- net VSSA: track 0.00 -> 50.4 mm, vias 0 -> 1
- net EXT1_G: track 0.00 -> 27.9 mm, vias 0 -> 2
- net Y_EN: track 11.3 -> 36.9 mm
- net DAT3: track 0.00 -> 25.1 mm
- net Y_DIR: track 9.30 -> 34.4 mm
- net Y_STEP: track 9.74 -> 34.8 mm
- net DAT2: track 0.00 -> 24.3 mm
- net CMD: track 0.00 -> 21.7 mm
- net VDDOUT: track 13.0 -> 34.2 mm, vias 0 -> 2
- net DAT0: track 0.00 -> 19.7 mm
- net ESP_RXD: track 0.00 -> 19.3 mm
- net CLK: track 0.00 -> 19.0 mm
- net ESP_TXD: track 0.00 -> 18.5 mm
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
Commit message: 20 parts left
Parts:
- added R51, R52, R53, R54, R55, R56: 10K, resistor:R0603
- C72, C73, C74: value (none) -> 2.2u
- moved C74 158.0 mm to (33.0, 42.5), turned to 270 degrees
- moved D6 148.9 mm to (29.5, 47.5), turned to 90 degrees
- moved C72 147.6 mm to (33.0, 34.0), turned to 270 degrees
- moved C73 143.1 mm to (33.0, 23.5), turned to 270 degrees
- moved D5 137.5 mm to (28.0, 39.5), turned to 90 degrees
- moved D4 127.5 mm to (34.0, 20.0), turned to 270 degrees
- moved R44 8.08 mm to (29.6, 36.6), turned to 180 degrees
- moved ERASE 7.81 mm to (81.0, 11.0)
- moved C29 2.12 mm to (58.5, 39.5)
- moved C25 1.00 mm to (78.0, 34.0)
- moved C30 1.00 mm to (55.5, 24.0)
- moved C17 0.71 mm to (64.6, 41.4)
- moved C23 0.71 mm to (79.5, 36.2)
- moved R14 0.71 mm to (81.0, 38.4)
- moved C19 0.50 mm to (62.0, 18.7)
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Connections:
- new net X_STOP_IN: R51.2, R56.1, X_STOP.1
- new net Y_STOP_IN: R52.2, R55.1, Y_STOP.1
- new net Z_STOP_IN: R53.2, R54.1, Z_STOP.1
- net +3V3: now also R54.2, R55.2, R56.2
- net EXT1: no longer IC3.24
- net FAN_PART: no longer IC3.21
- net X_DIR: now also IC3.21; no longer IC3.28
- net X_EN: now also IC3.24; no longer IC3.30
- net X_STEP: now also IC3.23; no longer IC3.29
- net X_STOP: now also IC3.30, R51.1; no longer IC3.73, X_STOP.1
- net Y_STOP: now also IC3.29, R52.1; no longer IC3.74, Y_STOP.1
- net Z_STOP: now also IC3.28, R53.1; no longer IC3.75, Z_STOP.1
Routing:
- net +3V3: track 325.3 -> 411.0 mm, vias 35 -> 36
- net E2_DIR: track 10.5 -> 90.4 mm, vias 0 -> 2
- net E2_STEP: track 10.6 -> 90.2 mm, vias 0 -> 2
- net E2_EN: track 10.6 -> 85.3 mm, vias 0 -> 2
- net E1_EN: track 12.0 -> 83.7 mm, vias 0 -> 4
- net E1_STEP: track 10.8 -> 77.8 mm, vias 0 -> 2
- net E1_DIR: track 10.7 -> 72.7 mm, vias 0 -> 2
- net X_STOP: track 0.00 -> 49.1 mm, vias 0 -> 2
- net Z_STOP: track 0.00 -> 43.3 mm, vias 0 -> 2
- net Y_STOP: track 0.00 -> 42.1 mm, vias 0 -> 2
- net VDDOUT: track 34.2 -> 70.8 mm, vias 2 -> 5
- net GND: track 1523.3 -> 1544.0 mm, vias 259 -> 260
- net X_DIR: track 12.2 -> 28.5 mm
- net X_STEP: track 12.3 -> 27.5 mm
- net MOT_MOSI: track 141.3 -> 156.3 mm, vias 5 -> 6
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