File: projects/AMR3350/V7-32/AMR3350.brd (EAGLE design)
At the start: 115 x 87 mm, 253 parts, among them IC1 A4403, IC10 TMC5130, IC11 TMC5130, IC12 74LS32D, IC13 TMC5130, IC2 LDO-TS1117CW-3V3, IC3 ATSAM4S8C, IC5 74HC125, IC6 74S08D, IC7 TMC5130, IC8 TMC5130, J1 MOLEX-105162-001, J2 MSTBV4, Q1 NX138BKS, Q2 NX138BKS, Q3 AON7524, Q4 AON7524, X2 12MHz

Commit message: 66 airwires left
Parts:
- removed IC6: 74S08D, 74xx-us:SO14
- added IC4: 74ABT125BQ, 74xx-us:DHVQFN14
- added R57: 4K7, resistor:R0603
- IC5: value 74HC125 -> 74AHC08; device misc:SO14 -> misc:DHVQFN14
- moved RESET 133.8 mm to (47.1, 31.6), turned to 270 degrees
- moved C44 117.8 mm to (35.1, 10.6), turned to 90 degrees
- moved C45 100.9 mm to (56.5, 9.70), turned to 180 degrees
- moved C16 92.0 mm to (54.0, 29.0), turned to 90 degrees
- moved IC5 88.8 mm to (56.5, 6.70), turned to 270 degrees
- moved C35 45.8 mm to (48.1, 25.6), turned to 180 degrees
- moved R16 43.2 mm to (48.1, 23.4), turned to 180 degrees
- moved C41 36.5 mm to (102.7, 43.0), turned to 270 degrees
- moved C43 34.5 mm to (94.8, 43.3), turned to 270 degrees
- moved C42 34.4 mm to (100.0, 43.0), turned to 270 degrees
- moved R38 34.3 mm to (102.7, 46.3), turned to 90 degrees
- moved R39 33.1 mm to (102.7, 49.6), turned to 90 degrees
- moved R37 32.2 mm to (100.0, 46.3), turned to 90 degrees
- moved R36 31.1 mm to (96.9, 44.2), turned to 90 degrees
- moved R40 30.8 mm to (100.0, 49.6), turned to 90 degrees
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Connections:
- net FAN_MOBO renamed FAN_3
- removed net FAN_E1: IC3.40, R42.1
- removed net FAN_E2: IC3.25, R43.1
- removed net FAN_PART: R45.1
- new net FAN_1: IC3.76, R42.1
- new net FAN_2: IC3.43, R43.1
- new net FAN_4: IC3.74, R45.1
- net +3V3: now also IC4.14; no longer IC5.14
- net +5V: now also IC5.14; no longer IC6.14
- net ENN: now also IC3.25; no longer IC3.71
- net ESP_DATA_RDY: now also IC3.73; no longer IC3.13
- net ESP_EN: now also IC3.71; no longer IC3.32
- net ESP_RESET: now also IC3.32; no longer IC3.43
- net EXT1: now also IC3.40
- net GND: now also IC4.1, IC4.10, IC4.13, IC4.2, IC4.7, IC5.2, IC5.EXP, R57.1; no longer IC5.12, IC5.13, IC5.4, IC6.10, IC6.7, IC6.9
- net LCD_BEEP: now also IC3.75, R57.2; no longer IC3.90
- net LCD_CS: now also IC5.10, IC5.12, IC5.5, IC5.9; no longer IC6.13, IC6.2, IC6.4, IC6.5
- net LCD_CS_BUF: now also IC5.8; no longer IC6.6
- net LCD_MISO: now also IC4.6; no longer IC5.8
- net LCD_MISO_BUF: now also IC4.5; no longer IC5.9
- net LCD_MOSI: now also IC4.9, IC5.4; no longer IC5.2, IC6.1
- net LCD_MOSI_BUF: now also IC5.6; no longer IC6.3
- net LCD_SCK: now also IC4.12, IC5.13; no longer IC5.5, IC6.12
- net LCD_SCK_BUF: now also IC5.11; no longer IC6.11
- net LCD_SD_CS: now also IC4.4; no longer IC5.10
- net SAM_TFR_RDY: now also IC3.72; no longer IC3.49
- net SD_MOSI_BUF: now also IC4.8; no longer IC5.3
- net SD_SCK_BUF: now also IC4.11; no longer IC5.6
- net SG_TST: now also IC3.49; no longer IC3.72
Routing:
- net GND: track 1544.0 -> 1864.8 mm, vias 260 -> 290
- net +5V: track 225.4 -> 345.5 mm, vias 6 -> 15
- net ESP_MOSI: track 5.42 -> 102.6 mm, vias 0 -> 4
- net ESP_SCK: track 4.04 -> 100.1 mm, vias 0 -> 4
- net ESP_RESET: track 0.00 -> 86.2 mm, vias 0 -> 2
- net ESP_NPCS0: track 0.00 -> 85.7 mm, vias 0 -> 2
- net MCDA2: track 0.00 -> 85.4 mm, vias 0 -> 2
- net ESP_MISO: track 0.00 -> 79.9 mm, vias 0 -> 2
- net ESP_UTXD: track 0.00 -> 76.4 mm, vias 0 -> 2
- net ESP_URXD: track 0.00 -> 72.4 mm, vias 0 -> 4
- net SAM_TFR_RDY: track 0.00 -> 70.1 mm, vias 0 -> 2
- net LCD_SD_CS: track 0.00 -> 69.6 mm, vias 0 -> 3
- net BED: track 0.00 -> 64.4 mm, vias 0 -> 4
- net +3V3: track 411.0 -> 475.2 mm, vias 36 -> 40
- net FAN_1: track 0.00 -> 64.1 mm, vias 0 -> 2
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
Commit message: Done!
Parts:
- removed C125, C128, C129, C130, C132: 100n, resistor:C0603
- removed C126: 4u7, resistor:C0603
- removed C127: 470n, resistor:C0603
- removed C131: 22n, resistor:C0603
- removed C133: 100u, resistor:PANASONIC_D
- removed C134, C135, C136, C137: 470p, resistor:C0402
- removed IC12: 74LS32D, 74xx-us:SO14
- removed R82, R83: 0R11, resistor:R1206
- removed R84: 20K, resistor:RTRIM3103
- removed R85: 20K, resistor:R0603
- added C112, C113, C84: 470p, resistor:C0402
- added C114: 100n, rcl:C0603
- added C75, C78, C79, C82, C83: 100n, resistor:C0603
- added C76: 470n, resistor:C0603
- added C77: 4u7, resistor:C0603
- added C80: 22n, resistor:C0603
- added C81: 100u, resistor:PANASONIC_D
- added IC9: TMC5130, TMC5130_3D_Printer_BOARD_V_2:QFP50P900X900X113-49N_NOFID
- added R66, R67: 0R11, resistor:R1206
- added R68: 20K, resistor:RTRIM3103
- added R69: 20K, resistor:R0603
- C100, C61, C87: value 470n -> 470p; device resistor:C0603 -> resistor:C0402
- C102, C50, C63, C89: value 100n -> 470n
- C103, C51, C64, C90: value 100n -> 4u7
- C104, C52, C65, C91: value 22n -> 100n
- C106, C54, C67, C93: value 100u -> 22n; device resistor:PANASONIC_D -> resistor:C0603
- C107, C55, C68, C94: value 470p -> 100u; device resistor:C0402 -> resistor:PANASONIC_D
- C108, C109, C56, C57, C69, C70, C95, C96: value 470p -> 100n; device resistor:C0402 -> resistor:C0603
- C111: value 100n -> 470p; device rcl:C0603 -> resistor:C0402
- C45, C46: value 100n -> 2.2u
- C47: value 4u7 -> 2.2u
- C48: value 470n -> 100n
- C59, C85, C98: value 100n -> 470p; device resistor:C0603 -> resistor:C0402
- C60, C86, C99: value 4u7 -> 470p; device resistor:C0603 -> resistor:C0402
- C72, C73, C74: value 2.2u -> 470p; device resistor:C0603 -> resistor:C0402
- IC11: value TMC5130 -> 74LS32D; device TMC5130_3D_Printer_BOARD_V_2:QFP50P900X900X113-49N_NOFID -> 74xx-us:SO14
- R39, R40, R41: value 4K7 0.1% -> 10K
- R42, R43, R44: value 1K -> 10K
- R45: value 1K -> 4K7 0.1%
- R46, R47: value 180R -> 4K7 0.1%
- R48, R49: value 4K7 -> 1K
- R50: value 180R -> 1K
- R51: value 10K -> 1K
- R52, R53, R56: value 10K -> 180R
- R54, R55: value 10K -> 4K7
- moved C69 95.6 mm to (109.8, 71.5), turned to 135 degrees
- moved C62 94.2 mm to (109.0, 61.9), turned to 0 degrees
- moved C47 93.6 mm to (35.1, 10.6)
- moved C73 93.4 mm to (109.1, 77.7), turned to 315 degrees
- moved C67 90.2 mm to (100.0, 72.3), turned to 45 degrees
- moved C68 87.1 mm to (95.5, 78.0), turned to 270 degrees
- moved C64 86.8 mm to (103.7, 74.3), turned to 90 degrees
- moved C71 84.0 mm to (99.5, 77.7)
- moved C72 81.4 mm to (101.7, 77.7)
- moved C66 81.0 mm to (97.6, 70.0), turned to 90 degrees
- moved C74 80.9 mm to (105.5, 78.5), turned to 180 degrees
- moved R62 80.8 mm to (97.3, 65.0)
- moved R63 80.8 mm to (111.7, 65.0)
- moved R65 80.8 mm to (103.9, 76.9)
- moved R64 80.5 mm to (107.4, 75.6), turned to 135 degrees
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- renumbered 3V3 to 3V1, IC13 to IC6, X2 to X1
Connections:
- net +12V: now also C104.2, C107.+, C108.1, C109.1, C52.2, C55.+, C56.1, C57.1, C65.2, C68.+, C69.1, C70.1, C78.2, C79.1, C81.+, C82.1, C83.1, C91.2, C94.+, C95.1, C96.1, IC9.21, IC9.39, IC9.40; no longer C101.2, C102.1, C103.1, C106.+, C128.2, C129.1, C130.1, C132.1, C133.+, C49.2, C50.1, C51.1, C54.+, C62.2, C63.1, C64.1, C67.+, C88.2, C89.1, C90.1, C93.+, IC11.21, IC11.39, IC11.40
- net +3V3: now also C101.1, C114.1, C47.1, C49.1, C62.1, C75.1, C88.1, IC11.14, IC9.10, R39.2, R40.2, R41.2; no longer C111.1, C125.1, C44.1, C46.1, C59.1, C85.1, C98.1, IC11.10, IC12.14, R54.2, R55.2, R56.2
- net +5V: now also C102.1, C50.1, C63.1, C76.1, C89.1, IC9.34, R69.2; no longer C100.1, C127.1, C45.1, C61.1, C87.1, IC11.34, R85.2
- net 5V_E1: now also C51.1; no longer C126.1
- net 5V_E2: now also C64.1; no longer C47.1
- net 5V_X: now also C77.1, IC8.33; no longer C86.1, IC10.33
- net 5V_Y: now also C90.1, IC9.33; no longer C99.1, IC11.33
- net 5V_Z: now also C103.1, IC10.33; no longer C60.1, IC8.33
- net A1_E1: now also C58.1; no longer C134.1
- net A1_E2: now also C71.1; no longer C55.1
- net A1_X: now also C84.1, IC8.46; no longer C94.1, IC10.46
- net A1_Y: now also C97.1, IC9.46; no longer C107.1, IC11.46
- net A1_Z: now also C110.1, IC10.46; no longer C68.1, IC8.46
- net A2_E1: now also C59.1; no longer C135.1
- net A2_E2: now also C72.1; no longer C56.1
- net A2_X: now also C85.1, IC8.42; no longer C95.1, IC10.42
- net A2_Y: now also C98.1, IC9.42; no longer C108.1, IC11.42
- net A2_Z: now also C111.1, IC10.42; no longer C69.1, IC8.42
- net ADVREF: now also R45.2, R46.2, R47.2; no longer R39.2, R40.2, R41.2
- net B1_E1: now also C60.1; no longer C136.1
- net B1_E2: now also C73.1; no longer C57.1
- net B1_X: now also C86.1, IC8.15; no longer C96.1, IC10.15
- net B1_Y: now also C99.1, IC9.15; no longer C109.1, IC11.15
- net B1_Z: now also C112.1, IC10.15; no longer C70.1, IC8.15
- net B2_E1: now also C61.1; no longer C137.1
- net B2_E2: now also C74.1; no longer C58.1
- net B2_X: now also C87.1, IC8.19; no longer C97.1, IC10.19
- net B2_Y: now also C100.1, IC9.19; no longer C110.1, IC11.19
- net B2_Z: now also C113.1, IC10.19; no longer C71.1, IC8.19
- net BED: now also R56.1; no longer R50.1
- net BED_L: now also R55.1; no longer R49.1
- net BED_OUT: now also R56.2; no longer R50.2
- net BRA_E1: now also R58.1; no longer R82.1
- net BRA_E2: now also R62.1; no longer R58.1
- net BRA_X: now also IC8.44, R66.1; no longer IC10.44, R70.1
- net BRA_Y: now also IC9.44, R70.1; no longer IC11.44, R74.1
- net BRA_Z: now also IC10.44, R74.1; no longer IC8.44, R62.1
- net BRB_E1: now also R59.1; no longer R83.1
- net BRB_E2: now also R63.1; no longer R59.1
- net BRB_X: now also IC8.17, R67.1; no longer IC10.17, R71.1
- net BRB_Y: now also IC9.17, R71.1; no longer IC11.17, R75.1
- net BRB_Z: now also IC10.17, R75.1; no longer IC8.17, R63.1
- net CPI_E1: now also C54.1; no longer C131.1
- net CPI_E2: now also C67.1; no longer C52.1
- net CPI_X: now also C80.1, IC8.37; no longer C91.1, IC10.37
- net CPI_Y: now also C93.1, IC9.37; no longer C104.1, IC11.37
- net CPI_Z: now also C106.1, IC10.37; no longer C65.1, IC8.37
- net CPO_E1: now also C54.2; no longer C131.2
- net CPO_E2: now also C67.2; no longer C52.2
- net CPO_X: now also C80.2, IC8.35; no longer C91.2, IC10.35
- net CPO_Y: now also C93.2, IC9.35; no longer C104.2, IC11.35
- net CPO_Z: now also C106.2, IC10.35; no longer C65.2, IC8.35
- net E1_FUSED: now also R54.2; no longer R48.2
- net E2_FUSED: now also R55.2; no longer R49.2
- net ENN: now also IC9.29; no longer IC11.29
- net EXT1: now also R52.1; no longer R46.1
- net EXT1_G: now also R52.2; no longer R46.2
- net EXT2: now also R53.1; no longer R47.1
- net EXT2_G: now also R53.2; no longer R47.2
- net EXT_L: now also R54.1; no longer R48.1
- net FAN1_G: now also R48.2; no longer R42.2
- net FAN2_G: now also R49.2; no longer R43.2
- net FAN3_G: now also R50.2; no longer R44.2
- net FAN4_G: now also R51.2; no longer R45.2
- net FAN_1: now also R48.1; no longer R42.1
- net FAN_2: now also R49.1; no longer R43.1
- net FAN_3: now also R50.1; no longer R44.1
- net FAN_4: now also R51.1; no longer R45.1
- net GND: now also C101.2, C104.1, C107.-, C112.2, C113.2, C114.2, C49.2, C52.1, C55.-, C62.2, C65.1, C68.-, C75.2, C76.2, C77.2, C78.1, C81.-, C82.2, C83.2, C84.2, C88.2, C91.1, C94.-, IC11.7, IC9.1, IC9.13, IC9.2, IC9.24, IC9.31, IC9.32, IC9.36, IC9.48, IC9.6, IC9.PAD, R66.2, R67.2, R68.1; no longer C101.1, C106.-, C107.2, C125.2, C126.2, C127.2, C128.1, C129.2, C130.2, C133.-, C134.2, C135.2, C136.2, C137.2, C49.1, C54.-, C55.2, C62.1, C67.-, C68.2, C88.1, C93.-, C94.2, IC11.1, IC11.13, IC11.2, IC11.24, IC11.31, IC11.32, IC11.36, IC11.48, IC11.6, IC11.PAD, IC12.7, R82.2, R83.2, R84.1
- net IREF_E1: now also R60.2; no longer R84.2
- net IREF_E2: now also R64.2; no longer R60.2
- net IREF_X: now also IC8.30, R68.2; no longer IC10.30, R72.2
- net IREF_Y: now also IC9.30, R72.2; no longer IC11.30, R76.2
- net IREF_Z: now also IC10.30, R76.2; no longer IC8.30, R64.2
- net MOT_MISO: now also IC9.7; no longer IC11.7
- net MOT_MOSI: now also IC9.5; no longer IC11.5
- net MOT_SCK: now also IC9.4; no longer IC11.4
- net REFIN_E1: now also R60.3, R61.1; no longer R84.3, R85.1
- net REFIN_E2: now also R64.3, R65.1; no longer R60.3, R61.1
- net REFIN_X: now also R68.3, R69.1; no longer R72.3, R73.1
- net REFIN_Y: now also R72.3, R73.1; no longer R76.3, R77.1
- net REFIN_Z: now also R76.3, R77.1; no longer R64.3, R65.1
- net SG_TST: now also IC11.6; no longer IC12.6
- net SG_TST_E1: now also IC11.12; no longer IC12.12
- net SG_TST_E1X: now also IC11.10, IC11.11; no longer IC12.10, IC12.11
- net SG_TST_E2: now also IC11.9; no longer IC12.9
- net SG_TST_EX: now also IC11.5, IC11.8; no longer IC12.5, IC12.8
- net SG_TST_X: now also IC11.13, IC8.27; no longer IC10.27, IC12.13
- net SG_TST_Y: now also IC11.1, IC9.27; no longer IC11.27, IC12.1
- net SG_TST_YZ: now also IC11.3, IC11.4; no longer IC12.3, IC12.4
- net SG_TST_Z: now also IC10.27, IC11.2; no longer IC12.2, IC8.27
- net T_BED: now also C46.1, R42.1; no longer C43.1, R36.1
- net T_BED_IN: now also R42.2, R47.1; no longer R36.2, R41.1
- net T_EXT1: now also C45.1, R43.1; no longer C42.1, R37.1
- net T_EXT2: now also C44.1, R44.1; no longer C41.1, R38.1
- net T_EXT_IN1: now also R43.2, R46.1; no longer R37.2, R40.1
- net T_EXT_IN2: now also R44.2, R45.1; no longer R38.2, R39.1
- net VCP_E1: now also C53.2; no longer C132.2
- net VCP_E2: now also C66.2; no longer C53.2
- net VCP_X: now also C79.2, IC8.38; no longer C92.2, IC10.38
- net VCP_Y: now also C92.2, IC9.38; no longer C105.2, IC11.38
- net VCP_Z: now also C105.2, IC10.38; no longer C66.2, IC8.38
- net X_DIR: now also IC8.9; no longer IC10.9
- net X_EN: now also IC8.3; no longer IC10.3
- net X_STEP: now also IC8.8; no longer IC10.8
- net X_STOP: now also C41.1, R36.1; no longer C73.1, R51.1
- net X_STOP_IN: now also R36.2, R39.1; no longer R51.2, R56.1
- net Y_DIR: now also IC9.9; no longer IC11.9
- net Y_EN: now also IC9.3; no longer IC11.3
- net Y_STEP: now also IC9.8; no longer IC11.8
- net Y_STOP: now also C42.1, R37.1; no longer C72.1, R52.1
- net Y_STOP_IN: now also R37.2, R40.1; no longer R52.2, R55.1
- net Z_DIR: now also IC10.9; no longer IC8.9
- net Z_EN: now also IC10.3; no longer IC8.3
- net Z_STEP: now also IC10.8; no longer IC8.8
- net Z_STOP: now also C43.1, R38.1; no longer C74.1, R53.1
- net Z_STOP_IN: now also R38.2, R41.1; no longer R53.2, R54.1
Routing:
- net +12V: track 425.8 -> 503.1 mm, vias 9 -> 18
- net EXT2: track 0.00 -> 65.0 mm, vias 0 -> 2
- net FAN_3: track 1.87 -> 59.3 mm, vias 1 -> 2
- net PWR_FAIL_DET2: track 2.32 -> 49.0 mm, vias 1 -> 2
- net GND: track 1864.8 -> 1908.0 mm, vias 290 -> 292
- net +3V3: track 475.2 -> 504.1 mm, vias 40 -> 42
- net +5V: track 345.5 -> 324.0 mm, vias 15 -> 12
- net SD_CD: track 61.1 -> 77.8 mm, vias 1 -> 2
- net E1_EN: track 85.0 -> 78.5 mm
- net E1_DIR: track 73.9 -> 78.2 mm
- net VDDOUT: track 71.8 -> 75.8 mm
- net EXT1_G: track 27.9 -> 24.0 mm
- net EXT1: track 39.0 -> 42.2 mm
- net LCD_SD_CS: track 69.6 -> 67.6 mm
- net MCDA3: track 55.7 -> 57.6 mm, vias 1 -> 2
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Other:
- board text added: "EE4SR3350"
- board text added: "Rev. 1.1.1"

Commit message: Final** version of AMRV7/EE4SR1.1.1, new APSR
Parts:
- renumbered 3V1 to +3V3, 5V to +5V, EXP_1 to EXP1, EXP_2 to EXP2
Routing:
- net +12V: track 503.1 -> 500.5 mm
- net FAN_1: track 64.1 -> 62.0 mm
- net SAM_TFR_RDY: track 70.1 -> 68.2 mm
- net GND: track 1908.0 -> 1906.6 mm
- net RESET: track 27.6 -> 26.3 mm
- net EXT2: track 65.0 -> 63.8 mm
- net ESP_DATA_RDY: track 49.6 -> 48.4 mm
- net USB_PWR_MON: track 26.5 -> 25.5 mm
- net LCD_SD_CS: track 67.6 -> 66.6 mm
- net FAN_2: track 60.6 -> 59.6 mm
- net Z_EN: track 71.0 -> 70.2 mm
- net Z_STEP: track 74.0 -> 73.3 mm
- net MCDA2: track 86.0 -> 85.3 mm
- net T_BED: track 31.7 -> 31.2 mm
- added copper zone on layer 1, net +12V
- added copper zone on layer 16, net +12V
- added copper zone on layer 16, net A1_E1
- added copper zone on layer 16, net A1_E2
- added copper zone on layer 16, net A1_X
- added copper zone on layer 16, net A1_Y
- added copper zone on layer 16, net A1_Z
- added copper zone on layer 16, net A2_E1
- added copper zone on layer 16, net A2_E2
- added copper zone on layer 16, net A2_X
- added copper zone on layer 16, net A2_Y
- added copper zone on layer 16, net A2_Z
- added copper zone on layer 16, net A_Z
- added copper zone on layer 16, net B1_E1
- added copper zone on layer 16, net B1_E2
- added copper zone on layer 16, net B1_X
- added copper zone on layer 16, net B1_Y
- added copper zone on layer 16, net B1_Z
- added copper zone on layer 16, net B2_E1
- added copper zone on layer 16, net B2_E2
- added copper zone on layer 16, net B2_X
- added copper zone on layer 16, net B2_Y
- added copper zone on layer 16, net B2_Z
- added copper zone on layer 16, net B_Z
- added copper zone on layer 16, net GND
Other:
- board text added: "+"
- board text added: "-"
- board text added: "1"
- board text added: "2"
- board text added: "3"
- board text added: "4"
- board text added: "BED"
- board text added: "Designed by Ethan Tillison"
- board text added: "E1"
- board text added: "E2"
- board text added: "ENDSTOPS"
- board text added: "FANS"
- board text added: "RESET"
- board text added: "S"
- board text added: "THERMISTORS"
- board text added: "USB"
- board text added: "X"
- board text added: "Y"
- board text added: "Z"
- board text added: "microSD"

Commit message: Cleaned up the EE4SR
Parts:
- moved ERASE 2.40 mm to (81.3, 12.1)
- moved R34 2.21 mm to (106.6, 37.9)
- moved C62 1.36 mm to (107.7, 61.5)
- moved C49 1.30 mm to (87.8, 61.4)
- moved C17 1.14 mm to (65.5, 40.7), turned to 180 degrees
- moved R48 1.08 mm to (32.4, 9.70)
- moved C40 1.03 mm to (93.3, 22.1), turned to 270 degrees
- moved C110 0.95 mm to (9.20, 67.7), turned to 270 degrees
- moved R32 0.71 mm to (96.4, 27.3), turned to 270 degrees
- moved C44 0.60 mm to (102.1, 43.0)
- moved R27 0.50 mm to (104.0, 37.5)
- moved R49 0.50 mm to (26.8, 13.7)
Routing:
- net GND: track 1906.6 -> 1896.4 mm
- net ESP_DATA_RDY: track 48.4 -> 45.2 mm
- net MOT_MISO: track 157.7 -> 154.7 mm
- net SAM_TFR_RDY: track 68.2 -> 65.3 mm
- net +3V3: track 503.8 -> 501.0 mm
- net LCD_MISO_BUF: track 14.6 -> 12.2 mm
- net ERASE: track 18.3 -> 15.9 mm
- net EXT1: track 42.3 -> 39.9 mm
- net +12V: track 500.5 -> 502.8 mm
- net MOT_SCK: track 156.0 -> 153.8 mm
- net MOT_MOSI: track 156.0 -> 154.0 mm
- net E2_DIR: track 90.9 -> 88.9 mm
- net T_EXT1: track 33.0 -> 31.0 mm
- net E2_STEP: track 90.6 -> 89.1 mm
- net MCCK: track 56.2 -> 54.8 mm
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- added copper zone on layer 1, net +5V
Other:
- board size 115 x 87 mm -> 116 x 87 mm

Commit message: Minor improvements, cam
Parts:
- moved R14 0.71 mm to (80.5, 37.9)
- moved C34 0.57 mm to (75.7, 36.4)
- moved C23 0.51 mm to (79.0, 36.3), turned to 135 degrees
- moved C33 0.20 mm to (77.7, 39.6)
- moved C22 0.14 mm to (81.4, 35.1)
Routing:
- net T_BED: track 29.9 -> 30.7 mm
- net +3V3: track 501.0 -> 501.7 mm
- net T_EXT2: track 34.6 -> 35.1 mm
- net GND: track 1896.4 -> 1896.0 mm, vias 292 -> 293
